File: BBB.sch (KiCad schematic (older format))
At the start: 29 parts, among them J3 addr, P19 U6_OE, P20 5V_LINK, P21 CONN_23X2, P22 CONN_23X2, Q5 2N7002KW, SW4 PWR_BBB, SW5 GPIO1_6, SW6 GPIO1_29, U10 BEAGLEBONE, U8 TSX0108, U9 CAT24C256

Commit message: uCm initial commit, work in progress
Parts:
- R15, R26, R27: symbol R_10K -> R
Changed lines of the file:
@@
 EESchema Schematic File Version 2
+LIBS:uCm
 LIBS:Conn-raspberry
 LIBS:power
-LIBS:uControl
-LIBS:uControl_v3-cache
-EELAYER 27 0
+LIBS:uCm-cache
+EELAYER 25 0
 EELAYER END
 $Descr A4 11693 8268
@@
 $EndComp
 $Comp
-L R_10K R15
+L R R15
 U 1 1 52A6192E
 P 2850 4525
@@
 	-1   0    0    -1
 $EndComp
-Text Notes 3125 5525 0    40   Italic 8
+Text Notes 3125 5625 0    40   Italic 8
 allows linking \nBBB 5V \nto uC_v3 5V
 Text Label 3125 5400 0    40   ~ 0
 5V0
-Text Notes 3150 4500 0    60   Italic 12
+Text Notes 3150 4700 0    60   Italic 12
 Enable/Disable U6\nfor comm betn\nBBB & uC_v3
 Text Label 2350 5075 0    40   ~ 0
@@
 $EndComp
 $Comp
-L R_10K R26
+L R R26
 U 1 1 52C03DD8
 P 2450 7150
@@
 $EndComp
 $Comp
-L R_10K R27
+L R R27
 U 1 1 52C03DF0
 P 3350 7150
@@
 Wire Notes Line
 	600  6600 600  4000
-Text Notes 650  4100 0    50   ~ 10
+Text Notes 650  4200 0    50   ~ 10
 LEVEL TRANSLATOR\nATMega (5V) <> BBB (3V3)
 Wire Notes Line
@@
 Wire Notes Line
 	600  7750 600  6700
-Text Notes 650  6800 0    50   ~ 10
+Text Notes 650  6875 0    50   ~ 10
 Discrete LEVEL TRANSLATOR\nATMega (5V) <> BBB (3V3)
-Text Notes 650  7000 0    40   ~ 8
+Text Notes 650  7150 0    40   ~ 8
 (can use for SPI Select\nbetn ATMega <> BBB)
 Wire Notes Line
@@
 Wire Notes Line
 	600  1000 1950 1000
-Text Notes 650  3700 0    50   ~ 10
+Text Notes 650  3775 0    50   ~ 10
 BBB Buttons\nGeneral purpose
 Text Notes 650  600  0    50   ~ 10
