File: interface.sch (KiCad schematic (older format))
At the start: 39 parts, among them M1 MANIFOLD, P10 C3SB, P11 VSel_Vlv, P14 X_VALVE, P15 Flow_Conn, P16 FLOWMETER, P17 PUMP, P18 Pump_Cable, P31 FLOW_CABLE, P34 VSel_Vlv2, P38 X_VALVE2, P7 GAGE_PR, P8 ABSO_PR, P9 C3SB, Q1 BCP5416TA, Q2 BCP5416TA, Q3 BCP5416TA, Q4 BCP5416TA, U1 TXB0104D

Commit message: uCm work in progress
Parts:
- removed C12, C14, C31, C5: 100nF, c_0805, symbol C
- removed D3, D9: S1D-13-F, diode-DO214AC, symbol D_1N4001
- removed P15: Flow_Conn, Conn_Flow_SFM3000_Male, symbol FLOWMETER
- removed P16: FLOWMETER, FlowMeter_SFM3000, symbol FLOWMETER
- removed P31: FLOW_CABLE, symbol FLOWMETER
- removed P34: VSel_Vlv2, Header_3, symbol CONN_3
- removed P38: X_VALVE2, X_Valve_2, symbol X_VALVE
- removed P8: ABSO_PR, HDIB002AUY8H5, symbol ABSO_PR
- removed Q3, Q4: BCP5416TA, SOT223, symbol NPN_TIP112G
- removed R6: 1k, r_0805, symbol R
- removed SP1: BUZZER, Speaker, symbol BUZZER
Connections:
- no-connect marks 21 -> 12
Other:
- note removed: "Connector at uC_v2"
- note removed: "Flow Meter cable"
- note removed: "Flow Meter, I2C , SFM3000\nAddress : 64 (h40)"
- note removed: "FlowMeter Footprint"
- note removed: "Pressure Sensor #2, Absolute, I2C Bus [HDIB002AUY8H5]"
- note removed: "Speaker, 5V DC\ndigital PWM port ~PD6"
- note removed: "Valve #2 on digital port PD4\neither 12V (V_IN) or 5V0"
