File: uCm.sch (KiCad schematic (older format))
At the start: 41 parts, among them P1 AREF, P23 Alt_Add, P28 Int1, P29 Int2, P4 ICSP, P5 FTDI, SW1 Reset, SW2 INT0, SW3 INT1, U11 ADXL345, U7 ATMEGA328-AU-ND, X1 16MHz

Commit message: uCm work in progress
Parts:
- added B13, B14: PB0, I_O, symbol I_O
- added B7: PC1, I_O, symbol I_O
Connections:
- net PC2_Pr2 renamed PC2
- net PC2: now also B7.1
- net PD4_Valve2 renamed PD4
- net PD4: now also B13.1
- net ~PD6_Spk renamed ~PD6
- net ~PD6: now also B14.1
Other:
- note added: "PUMP PWM"
- note added: "SW INT0"
- note added: "SW INT1"
- note removed: "Analog, from Absolute Pr Sensor"
- note removed: "Blank (ex Pulse)"
- note removed: "Blank (ex Pump PB0_IO_R)"
- note removed: "Blank (ex Pump PD7_IO_X)"
- note removed: "PUMP PWM (ex Pump ~PB1_IO_T)"
- note removed: "SW INT0 (ex Flow_Tx)"
- note removed: "SW INT1 (ex Blank)"
- note removed: "Speaker PWM (ex Blank)"
- note removed: "Valve #2 (ex Flow_Rx)"
Changed lines of the file:
@@
 $EndComp
 Text Notes 4550 3450 0    40   ~ 0
-SW INT1 (ex Blank)
+SW INT1
 $Comp
 L SCREW SC1
@@
 F10 "PC3_Pr1" I L 10050 3725 40
 F11 "3V3" B L 10050 1925 40
-F12 "SCL" I L 10050 3325 40
-F13 "SDA" I L 10050 3425 40
-F14 "PC2_Pr2" I L 10050 3625 40
-F15 "PD4_Valve2" I L 10050 2625 40
 F16 "~PB1_Pump" I L 10050 3125 40
-F17 "~PD6_Spk" I L 10050 2825 40
 $EndSheet
 NoConn ~ 8650 5825
-Text Label 9600 3625 0    40   ~ 0
-PC2_Pr2
-Text Label 9600 2825 0    40   ~ 0
-~PD6_Spk
-Text Label 9600 3425 0    40   ~ 0
-SDA
-Text Label 9600 3325 0    40   ~ 0
-SCL
 Text Label 9600 1925 0    40   ~ 0
 3V3
@@
 CS #1 Pr Sensor
 Text Notes 4550 4150 0    40   ~ 0
-PUMP PWM (ex Pump ~PB1_IO_T)
+PUMP PWM
 Text Notes 4550 4050 0    40   ~ 0
-Blank (ex Pump PB0_IO_R)
+Blank
 Text Notes 4550 3850 0    40   ~ 0
-Blank (ex Pump PD7_IO_X)
+Blank
 Text Notes 4550 3750 0    40   ~ 0
-Speaker PWM (ex Blank)
+Blank
 Text Notes 4550 3650 0    40   ~ 0
 Valve #1 PWM
 Text Notes 4550 3550 0    40   ~ 0
-Valve #2 (ex Flow_Rx)
+Blank
 Text Notes 4550 3350 0    40   ~ 0
-SW INT0 (ex Flow_Tx)
+SW INT0
 Text Label 9600 3125 0    40   ~ 0
 ~PB1_Pump
@@
 Text Label 9600 3725 0    40   ~ 0
 PC3_Pr1
-Text Label 9600 2625 0    40   ~ 0
-PD4_Valve2
 Text Label 9600 2725 0    40   ~ 0
 ~PD5_Valve
@@
 ~PD5_Valve
 Text Label 4125 3750 0    40   ~ 0
-~PD6_Spk
+~PD6
 Text Label 4125 3450 0    40   ~ 0
 ~PD3
@@
 PC1
 Text Label 4125 2450 0    40   ~ 0
-PC2_Pr2
+PC2
 Text Label 4125 2550 0    40   ~ 0
 PC3_Pr1
@@
 PD7
 Text Label 4125 3550 0    40   ~ 0
-PD4_Valve2
+PD4
 Text Label 4800 650  0    40   ~ 0
 5V0
@@
 $EndComp
 Text Notes 4550 2250 0    40   ~ 0
-Blank (ex Pulse)
+Blank
 Text Notes 4550 2350 0    40   ~ 0
 Blank
@@
 	7025 6300 8000 6300
 Wire Wire Line
-	9600 2825 10050 2825
-Wire Wire Line
-	9600 3325 10050 3325
-Wire Wire Line
 	9600 3125 10050 3125
 Wire Wire Line
 	9600 2725 10050 2725
-Wire Wire Line
-	9600 2625 10050 2625
 Wire Wire Line
 	9600 3725 10050 3725
@@
 	9600 1925 10050 1925
 Wire Wire Line
-	9600 3425 10050 3425
-Wire Wire Line
-	9600 3625 10050 3625
-Wire Wire Line
 	10050 825  9775 825
 Wire Notes Line
@@
 Connection ~ 975  2550
 Text Notes 4550 2450 0    40   ~ 0
-Analog, from Absolute Pr Sensor
+Blank
 Text Notes 4550 2550 0    40   ~ 0
 Analog, from Gage Pr Sensor
@@
 Wire Wire Line
 	7500 2975 7775 2975
+$Comp
+L I_O B7
+U 1 1 55A3A3EC
+P 4275 2450
+F 0 "B7" H 4355 2450 40  0000 L CNN
+F 1 "PC1" H 4275 2505 30  0001 C CNN
+F 2 "I_O" H 4275 2450 60  0001 C CNN
+F 3 "" H 4275 2450 60  0000 C CNN
+	1    4275 2450
+	1    0    0    -1
+$EndComp
+$Comp
+L I_O B13
+U 1 1 55A3A7AC
+P 4275 3550
+F 0 "B13" H 4355 3550 40  0000 L CNN
+F 1 "PB0" H 4275 3605 30  0001 C CNN
+F 2 "I_O" H 4275 3550 60  0001 C CNN
+F 3 "" H 4275 3550 60  0000 C CNN
+	1    4275 3550
+	1    0    0    -1
+$EndComp
+$Comp
+L I_O B14
+U 1 1 55A3B103
+P 4275 3750
+F 0 "B14" H 4355 3750 40  0000 L CNN
+F 1 "PB0" H 4275 3805 30  0001 C CNN
+F 2 "I_O" H 4275 3750 60  0001 C CNN
+F 3 "" H 4275 3750 60  0000 C CNN
+	1    4275 3750
+	1    0    0    -1
+$EndComp
 $EndSCHEMATC

Commit message: uCm KISS version
Parts:
- removed C42: 100uF, C_ELCO_SMD, symbol C_POL_1
- removed C43, C44: 100nF, c_0805, symbol C
- removed P23: Alt_Add, ShortLink2, symbol CONN_3
- removed P28: Int1, ShortLink2, symbol CONN_3
- removed P29: Int2, ShortLink2, symbol CONN_3
- removed U11: ADXL345, ADXL345, symbol ADXL345
Connections:
- no-connect marks 3 -> 1
Other:
- note removed: "Accelerometer, 3V3 I2C"
