File: KiCAD/uCm.kicad_pcb (KiCad board)
At the start: 2 copper layers, 190 x 152 mm, 149 parts, among them J1 5V_EXT, J2 3V3_EXT, J3 addr, P1 AREF, P10 C3SB, P11 VSel_Vlv, P13 PWR_IN, P14 X_VALVE, P15 Flow_Conn, P16 FLOWMETER, P17 PUMP, P19 U6_OE, P20 5V_LINK, P21 CONN_23X2, P22 CONN_23X2, P23 Alt_Add, P24 PWR_IN, P28 Int1, P29 Int2, P34 VSel_Vlv2, P38 X_VALVE2, P4 ICSP, P5 FTDI, P7 GAGE_PR, P8 ABSO_PR, P9 C3SB, Q1 BCP5416TA, Q2 BCP5416TA, Q3 BCP5416TA, Q4 BCP5416TA, Q5 2N7002KW, SW1 Reset, SW2 INT0, SW3 INT1, SW4 PWR_BBB, SW5 GPIO1_6, SW6 GPIO1_29, U1 TXB0104D, U10 BEAGLEBONE, U11 ADXL345, U3 TPS62133, U4 TPS62132, U5 DS3231N, U7 ATMEGA328-AU-ND, U8 TSX0108, U9 CAT24C256, X1 16MHz

Commit message: work in progress
Parts:
- removed B5: 5V_ATMega, I_O
- removed B6: 3V3_BBB, I_O
- removed C12, C39, C40, C41, C43, C44, C5: 100nF, c_0805
- removed C42: 100uF, C_ELCO_SMD
- removed J3: addr, Header_2x2
- removed P19: U6_OE, ShortLink2
- removed P20: 5V_LINK, ShortLink2
- removed P23: Alt_Add, ShortLink2
- removed P28: Int1, ShortLink2
- removed P29: Int2, ShortLink2
- removed PCB1: PCB, PCB
- removed Q5: 2N7002KW, SOT323
- removed R12: 4k7, r_0805
- removed R15, R26, R27: 10k, r_0805
- removed R16, R17, R18, R23: 4k75, r_0805
- removed R19, R20: 1k5, r_0805
- removed R24, R25: 220, r_0805
- removed SW4: PWR_BBB, SW_PB_V_H
- removed SW5: GPIO1_6, SW_PB_V_H
- removed SW6: GPIO1_29, SW_PB_V_H
- removed U11: ADXL345, ADXL345
- removed U8: TSX0108, TXS0108EPWR
- removed U9: CAT24C256, SO8E
- added B7: PC1, uCm:I_O, F.Cu at (106.9, 181.4)
- added G1: Logo_Wyolum, uCm:Logo-WL3, F.Cu at (124.7, 179.5)
- added G2: Logo_Wyolum, uCm:Logo-WL3, F.Cu at (115.5, 181.6)
- B1, B10, B11, B12, B2, B3, B4, B8, B9: footprint I_O -> uCm:I_O
- BT1: footprint CR2032 -> uCm:CR2032
- C1, C10, C11, C13, C14, C17, C18, C20, C21, C23, C28, C29, C31, C32, C34, C35, C4, C7, C8, C9: footprint c_0805 -> uCm:c_0805
- C19, C33: footprint c_1210 -> uCm:C_1210
- C2, C3: footprint c_0603 -> uCm:c_0603
- C22, C26, C27, C36, C37: footprint C_ELCO_SMD -> uCm:C_ELCO_SMD
- C30, C38: footprint c_1206 -> uCm:C_1206
- D1, D3, D4, D9: footprint diode-DO214AC -> uCm:diode-DO214AC
- D5, D6, D7, D8: footprint led_0805 -> uCm:led_0805
- G3, G4: footprint OSHW_6mm -> uCm:OSHW_6mm
- J1, J2, P13: footprint Header_2 -> uCm:Header_2
- L1, L2: footprint Inductor_SMD3 -> uCm:Inductor_SMD3
- P1: footprint ShortLink2 -> uCm:ShortLink2
- P10, P9: footprint pin_strip_4-90 -> uCm:pin_strip_4-90
- P11, P34: footprint Header_3 -> uCm:Header_3
- P14, P38: footprint X_Valve_2 -> uCm:X_Valve_2
- P17: footprint Pump_P54E01R_02 -> uCm:Pump_P54E01R_02
- P24: footprint JACK_ALIM -> uCm:JACK_ALIM
- P4: footprint Header_ISP -> uCm:Header_ISP
- P5: footprint Header_FTDI -> uCm:Header_FTDI
- P7: footprint HCEM500GUH9P3 -> uCm:HCEM500GUH9P3
- Q1, Q2, Q3, Q4: footprint SOT223 -> uCm:SOT223
- R1, R10, R11, R13, R14, R2, R21, R22, R3, R4, R5, R6, R7, R8, R9: footprint r_0805 -> uCm:r_0805
- SC1, SC10, SC2, SC3, SC4, SC5, SC6, SC7, SC8, SC9: footprint vite_3mm -> uCm:vite_3mm
- SP1: footprint Speaker -> uCm:Speaker
- SW1, SW2, SW3: footprint SW_PB_V_H -> uCm:SW_PB_V_H
- U1: footprint TXB0104D -> uCm:TXB0104D
- U3, U4: footprint TPS62132 -> uCm:TPS62132
- U5: footprint DS3231 -> uCm:DS3231
- U7: footprint TQFP32 -> uCm:TQFP32
- X1: footprint Xtal_SMD3 -> uCm:Xtal_SMD3
- moved C30 0.06 mm to (174.0, 152.1), turned to 90 degrees
- moved C38 0.06 mm to (151.0, 152.1), turned to 90 degrees
- turned C19 to 270 degrees
- turned C33 to 270 degrees
Connections:
- net /BBB/MISO renamed /Interface/MISO
- net /BBB/RESET renamed /RESET
- net /BBB/RXD renamed /RXD
- net /BBB/SCK renamed /Interface/SCK
- net /BBB/TXD renamed /TXD
- net /BBB/~MOSI renamed /Interface/~MOSI
- C1 pad 1: /BBB/5V0 -> /Interface/5V0
- C11 pad 1: /BBB/5V0 -> /Interface/5V0
- C14 pad 1: /BBB/5V0 -> /Interface/5V0
- C18 pad 2: /BBB/5V0 -> /Interface/5V0
- C19 pad 1: /BBB/5V0 -> /Interface/5V0
- C28 pad 1: /BBB/5V0 -> /Interface/5V0
- C7 pad 1: /BBB/5V0 -> /Interface/5V0
- C9 pad 1: /BBB/5V0 -> /Interface/5V0
- D3 pad 2: /BBB/5V0 -> /Interface/5V0
- J1 pad 1: /BBB/5V0 -> /Interface/5V0
- L1 pad 2: /BBB/5V0 -> /Interface/5V0
- P1 pad 3: /BBB/5V0 -> /Interface/5V0
- P10 pad 1: /BBB/5V0 -> /Interface/5V0
- P10 pad 2: /BBB/SCL -> /Interface/SCL
- P10 pad 3: /BBB/SDA -> /Interface/SDA
- P11 pad 1: /BBB/5V0 -> /Interface/5V0
- P34 pad 1: /BBB/5V0 -> /Interface/5V0
- P4 pad 2: /BBB/5V0 -> /Interface/5V0
- P8 pad 2: /Interface/PC2_Pr2 -> (no net)
- P9 pad 1: /BBB/5V0 -> /Interface/5V0
- P9 pad 2: /BBB/SCL -> /Interface/SCL
- P9 pad 3: /BBB/SDA -> /Interface/SDA
- R1 pad 1: /BBB/5V0 -> /Interface/5V0
- R11 pad 1: /BBB/5V0 -> /Interface/5V0
- R2 pad 1: /BBB/5V0 -> /Interface/5V0
- R2 pad 2: /BBB/SDA -> /rtc/SDA
- R3 pad 1: /BBB/5V0 -> /Interface/5V0
- R3 pad 2: /BBB/SCL -> /rtc/SCL
- R5 pad 1: /BBB/5V0 -> /Interface/5V0
- R6 pad 1: /BBB/5V0 -> /Interface/5V0
- R7 pad 2: /BBB/5V0 -> /Interface/5V0
- R8 pad 1: /BBB/5V0 -> /Interface/5V0
- SP1 pad 1: /BBB/5V0 -> /Interface/5V0
- SW2 pad 2: /BBB/5V0 -> /Interface/5V0
- SW3 pad 2: /BBB/5V0 -> /Interface/5V0
- U1 pad 14: /BBB/5V0 -> /Interface/5V0
- U3 pad 14: /BBB/5V0 -> /Interface/5V0
- U5 pad 15: /BBB/SDA -> /rtc/SDA
- U5 pad 16: /BBB/SCL -> /rtc/SCL
- U5 pad 2: /BBB/5V0 -> /Interface/5V0
- U7 pad 18: /BBB/5V0 -> /Interface/5V0
- U7 pad 25: /Interface/PC2_Pr2 -> /PC2
- U7 pad 27: /BBB/SDA -> /rtc/SDA
- U7 pad 28: /BBB/SCL -> /rtc/SCL
- U7 pad 4: /BBB/5V0 -> /Interface/5V0
- U7 pad 6: /BBB/5V0 -> /Interface/5V0
Routing:
- net /BBB/5V0: track 593.2 -> 43.1 mm, vias 10 -> 4
- net /Interface/5V0: track 0.00 -> 379.8 mm, vias 0 -> 4
- net GND: track 1144.0 -> 895.8 mm, vias 18 -> 16
- net /BBB/VDD_3V3EXP: track 219.5 -> 8.15 mm, vias 3 -> 0
- net /BBB/SDA: track 194.8 -> 11.2 mm, vias 4 -> 0
- net /BBB/SCL: track 179.3 -> 20.1 mm, vias 2 -> 0
- net /BBB/I2C1_SCL: track 154.3 -> 5.61 mm, vias 1 -> 0
- net /BBB/I2C1_SDA: track 152.0 -> 5.61 mm, vias 2 -> 0
- net /BBB/TIMER6: track 126.1 -> 5.61 mm, vias 2 -> 0
- net +3.3V: track 366.9 -> 248.6 mm, vias 7 -> 6
- net /BBB/BBB_OE: track 80.1 -> 0.00 mm, vias 2 -> 0
- net /BBB/SPI1_D0: track 77.6 -> 5.61 mm, vias 1 -> 0
- net /BBB/SPI1_SCLK: track 77.1 -> 5.61 mm, vias 1 -> 0
- net /BBB/UART1_RXD: track 74.0 -> 5.61 mm, vias 1 -> 0
- net /BBB/UART1_TXD: track 73.5 -> 5.61 mm
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