File: KiCAD/uCm.kicad_pcb (KiCad board)
At the start: 2 copper layers, 190 x 152 mm, 116 parts, among them J1 5V_EXT, J2 3V3_EXT, P1 AREF, P10 C3SB, P11 VSel_Vlv, P13 PWR_IN, P14 X_VALVE, P15 Flow_Conn, P16 FLOWMETER, P17 PUMP, P21 CONN_23X2, P22 CONN_23X2, P24 PWR_IN, P34 VSel_Vlv2, P38 X_VALVE2, P4 ICSP, P5 FTDI, P7 GAGE_PR, P8 ABSO_PR, P9 C3SB, Q1 BCP5416TA, Q2 BCP5416TA, Q3 BCP5416TA, Q4 BCP5416TA, SW1 Reset, SW2 INT0, SW3 INT1, U1 TXB0104D, U10 BEAGLEBONE, U3 TPS62133, U4 TPS62132, U5 DS3231N, U7 ATMEGA328-AU-ND, X1 16MHz

Commit message: making some progress on the PCB
Parts:
- removed G1, G2: Logo_Wyolum, uCm:Logo-WL3
- removed G3, G4: Logo_OH, uCm:OSHW_6mm
- removed P15: Flow_Conn, Conn_Flow_SFM3000_Male
- removed P16: FLOWMETER, FlowMeter_SFM3000
- removed P21, P22: CONN_23X2, PIN_ARRAY_23X2
- removed P8: ABSO_PR, HDIB002AUY8H5
- removed SC1, SC2, SC5, SC8: SCREW, uCm:vite_3mm
- removed U10: BEAGLEBONE, BEAGLEBONE
- moved D9 159.4 mm to (188.0, 102.0), turned to 270 degrees
- moved P38 151.1 mm to (182.0, 102.0), turned to 180 degrees
- moved Q3 149.8 mm to (195.0, 102.0)
- moved C31 147.1 mm to (195.0, 106.9), turned to 180 degrees
- moved P34 145.2 mm to (202.5, 101.9), turned to 90 degrees
- moved D1 98.5 mm to (145.0, 102.0), turned to 270 degrees
- moved SC3 90.5 mm to (115.0, 52.0)
- moved B7 87.7 mm to (175.0, 126.0)
- moved P14 87.7 mm to (139.0, 102.0), turned to 180 degrees
- moved C13 85.9 mm to (151.0, 107.0), turned to 180 degrees
- moved Q1 85.1 mm to (151.0, 102.0)
- moved P11 75.3 mm to (158.0, 102.0), turned to 90 degrees
- moved C10 54.9 mm to (131.0, 118.0), turned to 90 degrees
- moved P7 47.0 mm to (123.0, 122.0)
- moved SP1 45.6 mm to (118.0, 155.0), turned to 0 degrees
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Connections:
- P17 pad 3: (no net) -> Net-(P17-Pad3)
- P17 pad 5: (no net) -> Net-(P17-Pad5)
- P5 pad 3: (no net) -> Net-(P5-Pad3)
- P7 pad 7: (no net) -> Net-(P7-Pad7)
- U1 pad 6: (no net) -> Net-(U1-Pad6)
- U1 pad 9: (no net) -> Net-(U1-Pad9)
Routing:
- net GND: track 895.8 -> 0.00 mm, vias 16 -> 0
- net /Interface/12V: track 396.6 -> 0.00 mm, vias 2 -> 0
- net /Interface/5V0: track 379.8 -> 0.00 mm, vias 4 -> 0
- net +3.3V: track 248.6 -> 0.00 mm, vias 6 -> 0
- net /RESET: track 172.8 -> 0.00 mm, vias 1 -> 0
- net /Interface/PD4_Valve2: track 129.7 -> 0.00 mm, vias 2 -> 0
- net /Interface/~PD5_Valve: track 128.6 -> 0.00 mm, vias 2 -> 0
- net /Interface/PC3_Pr1: track 116.4 -> 0.00 mm, vias 2 -> 0
- net /Interface/SCK: track 108.2 -> 0.00 mm, vias 6 -> 0
- net /Interface/~PB1_Pump: track 103.4 -> 0.00 mm, vias 2 -> 0
- net /Interface/+Vlv: track 101.9 -> 0.00 mm
- net /PD2: track 89.5 -> 0.00 mm, vias 2 -> 0
- net /~PD3: track 87.3 -> 0.00 mm
- net /Interface/MISO: track 85.0 -> 0.00 mm, vias 4 -> 0
- net /TXD: track 77.7 -> 0.00 mm, vias 2 -> 0
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- removed copper zone on F.Cu, net /Interface/-Vlv
- removed copper zone on F.Cu, net /Interface/-Vlv2
- removed copper zone on B.Cu, net GND
- removed copper zone on F.Cu, net Net-(C17-Pad2)
Other:
- board size 190 x 152 mm -> 99 x 122 mm
- board text removed: "12V"
- board text removed: "3V3"
- board text removed: "3V3|D0|GND"
- board text removed: "3V3|OE|GND"
- board text removed: "5V0"
- board text removed: "5V0<>3V3"
- board text removed: "5V0|SCL|SDA|GND"
- board text removed: "A0"
- board text removed: "A1"
- board text removed: "GND|INT1|3V3"
- board text removed: "GND|INT2|3V3"
- board text removed: "ON<>OFF"
- board text removed: "RST SQW 32k"
- board text removed: "RTC"
- board text removed: "SDA|GND|5V0|SCL"
- board text removed: "uControl_v3"
- board text removed: "www.wyolum.com"
- board text removed: "wyolum.com"

Commit message: layout, work in progress
Parts:
- removed SC3, SC4: SCREW, uCm:vite_3mm
- P17: footprint uCm:Pump_P54E01R_02 -> uCm:Pump_P54E01R_03
- moved C31 153.6 mm to (49.0, 59.0), turned to 0 degrees
- moved P34 151.8 mm to (55.5, 64.0)
- moved Q3 150.9 mm to (49.0, 64.0)
- moved D9 149.9 mm to (43.0, 64.0)
- moved P38 149.9 mm to (37.0, 64.0)
- moved D7 143.3 mm to (16.0, 84.5), turned to 0 degrees
- moved D5 143.0 mm to (16.0, 81.5), turned to 0 degrees
- moved D6 142.8 mm to (16.0, 78.5), turned to 0 degrees
- moved D8 142.6 mm to (16.0, 75.5), turned to 0 degrees
- moved R5 138.7 mm to (58.5, 36.0), turned to 90 degrees
- moved R10 137.9 mm to (20.0, 84.5), turned to 0 degrees
- moved R8 137.5 mm to (20.0, 81.5), turned to 0 degrees
- moved R9 137.3 mm to (20.0, 78.5), turned to 0 degrees
- moved R13 137.1 mm to (20.0, 75.5), turned to 0 degrees
- moved C8 135.6 mm to (37.5, 25.0)
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Other:
- board size 99 x 122 mm -> 99 x 80 mm
- board text removed: "[+]"
- board text removed: "[+][-]"

Commit message: layout, work in progress
Parts:
- added G1: Logo_Wyolum, uCm:Logo-WL3, B.Cu at (95.5, 77.6)
- added G2: Logo_Wyolum, uCm:Logo-WL3, F.Cu at (83.4, 77.6)
- added G3: Logo_OH, uCm:OSHW_6mm, F.Cu at (89.8, 88.1)
- added G4: Logo_OH, uCm:OSHW_6mm, B.Cu at (89.8, 88.1)
- added REF**: via01, uCm:via_th, F.Cu at (28.2, 71.1)
- added REF**: via01, uCm:via_th, F.Cu at (72.5, 33.7)
- added REF**: via01, uCm:via_th, F.Cu at (89.1, 36.3)
- added REF**: via01, uCm:via_th, F.Cu at (81.9, 36.3)
- added REF**: via01, uCm:via_th, F.Cu at (97.4, 28.0)
- added REF**: via01, uCm:via_th, F.Cu at (87.4, 28.0)
- added REF**: via01, uCm:via_th, F.Cu at (83.7, 24.4)
- added REF**: via01, uCm:via_th, F.Cu at (52.2, 44.6)
- added REF**: via01, uCm:via_th, F.Cu at (52.2, 56.1)
- added REF**: via01, uCm:via_th, F.Cu at (53.5, 92.7)
- added REF**: via01, uCm:via_th, F.Cu at (79.6, 92.6)
- added REF**: via01, uCm:via_th, F.Cu at (58.8, 44.7)
- added REF**: via01, uCm:via_th, F.Cu at (69.0, 92.6)
- added REF**: via01, uCm:via_th, F.Cu at (41.8, 78.3)
- added REF**: via01, uCm:via_th, F.Cu at (82.0, 62.5)
- added REF**: via01, uCm:via_th, F.Cu at (69.3, 62.7)
- added REF**: via01, uCm:via_th, F.Cu at (43.0, 92.7)
- added REF**: via01, uCm:via_th, F.Cu at (18.6, 81.4)
- added REF**: via01, uCm:via_th, F.Cu at (54.0, 64.0)
- added REF**: via01, uCm:via_th, F.Cu at (65.8, 61.8)
- added REF**: via01, uCm:via_th, F.Cu at (40.6, 39.9)
- added REF**: via01, uCm:via_th, F.Cu at (44.8, 24.1)
- added REF**: via01, uCm:via_th, F.Cu at (77.5, 57.5)
- added REF**: via01, uCm:via_th, F.Cu at (35.6, 24.1)
- added REF**: via01, uCm:via_th, F.Cu at (27.3, 26.0)
- added REF**: via01, uCm:via_th, F.Cu at (39.3, 24.1)
- added REF**: via01, uCm:via_th, F.Cu at (58.8, 56.2)
- added REF**: via01, uCm:via_th, F.Cu at (80.5, 66.8)
- added REF**: via01, uCm:via_th, F.Cu at (91.8, 66.8)
- added REF**: via01, uCm:via_th, F.Cu at (82.0, 45.2)
- added REF**: via01, uCm:via_th, F.Cu at (83.9, 45.8)
- added REF**: via01, uCm:via_th, F.Cu at (80.1, 45.8)
- added REF**: via01, uCm:via_th, F.Cu at (60.0, 69.0)
- moved R2 87.4 mm to (96.8, 34.5), turned to 0 degrees
- moved R3 82.9 mm to (96.8, 37.2), turned to 0 degrees
- moved C14 78.0 mm to (18.6, 84.0), turned to 270 degrees
- moved D8 74.7 mm to (90.2, 67.0), turned to 270 degrees
- moved D5 73.0 mm to (87.5, 67.0), turned to 270 degrees
- moved R6 72.3 mm to (21.1, 84.0), turned to 270 degrees
- moved P10 72.2 mm to (85.0, 35.8), turned to 90 degrees
- moved P9 71.6 mm to (92.2, 35.8), turned to 90 degrees
- moved R13 70.4 mm to (90.2, 70.8), turned to 270 degrees
- moved D6 69.7 mm to (84.8, 67.0), turned to 270 degrees
- moved R8 68.4 mm to (87.5, 70.8), turned to 270 degrees
- moved D7 68.3 mm to (82.0, 67.0), turned to 270 degrees
- moved D3 68.3 mm to (24.3, 84.0), turned to 270 degrees
- moved R9 65.2 mm to (84.8, 70.8), turned to 270 degrees
- moved C11 64.4 mm to (82.8, 38.8), turned to 270 degrees
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Connections:
- C1 pad 1: /Interface/5V0 -> /AREF
- P14 pad 1: /Interface/+Vlv -> /Interface/-Vlv
- P14 pad 2: /Interface/-Vlv -> /Interface/+Vlv
- P17 pad 3: Net-(P17-Pad3) -> (no net)
- P17 pad 5: Net-(P17-Pad5) -> (no net)
- P38 pad 1: /Interface/+Vlv2 -> /Interface/-Vlv2
- P38 pad 2: /Interface/-Vlv2 -> /Interface/+Vlv2
- P5 pad 3: Net-(P5-Pad3) -> (no net)
- P7 pad 7: Net-(P7-Pad7) -> (no net)
- Q1 pad 1: /Interface/~PD5_Valve -> /Interface/PD4_Valve2
- Q3 pad 1: /Interface/PD4_Valve2 -> /Interface/~PD5_Valve
- R2 pad 2: /rtc/SDA -> /Interface/SDA
- R3 pad 2: /rtc/SCL -> /Interface/SCL
- U1 pad 6: Net-(U1-Pad6) -> (no net)
- U1 pad 9: Net-(U1-Pad9) -> (no net)
- U5 pad 15: /rtc/SDA -> /Interface/SDA
- U5 pad 16: /rtc/SCL -> /Interface/SCL
- U7 pad 27: /rtc/SDA -> /Interface/SDA
- U7 pad 28: /rtc/SCL -> /Interface/SCL
Routing:
- net /Interface/5V0: track 0.00 -> 402.5 mm, vias 0 -> 3
- net GND: track 0.00 -> 323.2 mm
- net /Interface/12V: track 0.00 -> 284.9 mm, vias 0 -> 1
- net +3.3V: track 0.00 -> 165.1 mm, vias 0 -> 3
- net /RESET: track 0.00 -> 112.0 mm
- net /Interface/SCK: track 0.00 -> 108.2 mm, vias 0 -> 2
- net /Interface/MISO: track 0.00 -> 102.7 mm, vias 0 -> 2
- net /Interface/~MOSI: track 0.00 -> 93.3 mm, vias 0 -> 2
- net /Interface/PC3_Pr1: track 0.00 -> 83.5 mm, vias 0 -> 2
- net /PD2: track 0.00 -> 78.5 mm, vias 0 -> 1
- net /~PD3: track 0.00 -> 67.7 mm
- net /Interface/~SS: track 0.00 -> 67.4 mm, vias 0 -> 2
- net /RXD: track 0.00 -> 66.8 mm, vias 0 -> 1
- net /TXD: track 0.00 -> 65.8 mm, vias 0 -> 1
- net /rtc/BAT: track 0.00 -> 57.6 mm, vias 0 -> 1
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- added copper zone on B.Cu, net GND

Commit message: layout, work in progress
Parts:
- added REF**: via01, uCm:via_th, F.Cu at (67.8, 78.3)
- added REF**: via01, uCm:via_th, F.Cu at (46.8, 92.7)
- added REF**: via01, uCm:via_th, F.Cu at (51.2, 79.6)
- added REF**: via01, uCm:via_th, F.Cu at (41.9, 81.0)
- added REF**: via01, uCm:via_th, F.Cu at (49.0, 80.1)
- added REF**: via01, uCm:via_th, F.Cu at (46.5, 78.5)
- added REF**: via01, uCm:via_th, F.Cu at (46.5, 80.1)
- added REF**: via01, uCm:via_th, F.Cu at (88.3, 78.2)
- added REF**: via01, uCm:via_th, F.Cu at (88.3, 81.2)
- added REF**: via01, uCm:via_th, F.Cu at (61.8, 81.2)
- added REF**: via01, uCm:via_th, F.Cu at (61.8, 78.2)
- added REF**: via01, uCm:via_th, F.Cu at (77.2, 79.6)
- added REF**: via01, uCm:via_th, F.Cu at (75.0, 80.1)
- added REF**: via01, uCm:via_th, F.Cu at (72.5, 78.5)
- added REF**: via01, uCm:via_th, F.Cu at (72.5, 80.1)
- added REF**: via01, uCm:via_th, F.Cu at (67.8, 81.0)
- added REF**: via01, uCm:via_th, F.Cu at (75.8, 92.6)
- added REF**: via01, uCm:via_th, F.Cu at (72.8, 92.6)
- added REF**: via01, uCm:via_th, F.Cu at (49.8, 92.7)
- moved G1 32.2 mm to (64.2, 85.5)
- moved G2 30.2 mm to (54.2, 85.5)
- moved REF** 24.3 mm to (40.1, 92.7)
- moved C14 20.8 mm to (38.2, 90.8), turned to 90 degrees
- moved R6 17.4 mm to (38.2, 87.0)
- moved D3 11.8 mm to (35.8, 87.0)
- moved Q4 5.31 mm to (35.8, 78.5)
- moved SP1 5.10 mm to (27.5, 87.0)
- moved REF** 5.03 mm to (31.5, 74.9)
- moved G3 4.07 mm to (85.8, 88.5)
- moved G4 4.07 mm to (85.8, 88.5)
- moved REF** 2.55 mm to (60.5, 46.6)
Connections:
- net Net-(C17-Pad2) renamed /Interface/Pump_Ret
Routing:
- net +3.3V: track 165.1 -> 195.3 mm
- net /Interface/5V0: track 402.5 -> 427.7 mm
- net /Interface/12V: track 284.9 -> 275.9 mm
- net GND: track 323.2 -> 316.1 mm
- net /RXD: track 66.8 -> 73.4 mm
- net /TXD: track 65.8 -> 71.1 mm
- net /RESET: track 112.0 -> 108.8 mm
- net /rtc/BAT: track 57.6 -> 60.1 mm
- net /Interface/Pump: track 26.9 -> 29.3 mm
- net /Interface/MISO: track 102.7 -> 100.7 mm
- net /Interface/~MOSI: track 93.3 -> 91.3 mm
- net /Interface/Spk: track 28.4 -> 26.5 mm
- net /PD2: track 78.5 -> 79.3 mm
- net /Interface/SCK: track 108.2 -> 107.5 mm
- net /Interface/~PD6_Spk: track 34.7 -> 35.3 mm
- added copper zone on F.Cu, net /Interface/-Vlv
- added copper zone on F.Cu, net /Interface/-Vlv2
- added copper zone on F.Cu, net /Interface/Pump_Ret
- added copper zone on F.Cu, net /Interface/Spk
- added copper zone on F.Cu, net GND
Other:
- board text added: "12V"
- board text added: "5V0|SCL|SDA|GND"
- board text added: "5V<>12V"
- board text added: "5V<>3V"
- board text added: "[-] [+]"
- board text added: "[-][+]"

Commit message: Board layout complete. Gerbers, PDF', BoM generated.
Parts:
- moved SP1 7.29 mm to (24.8, 80.2), turned to 0 degrees
- moved REF** 2.21 mm to (58.8, 45.2)
- moved G1 0.50 mm to (64.2, 85.0)
- moved G2 0.50 mm to (54.2, 85.0)
Routing:
- net /Interface/5V0: track 427.7 -> 443.7 mm
- net /Interface/Spk: track 26.5 -> 13.1 mm
- net /Interface/~MOSI: track 91.3 -> 90.7 mm
- net /TXD: track 71.1 -> 71.6 mm
- net /Interface/MISO: track 100.7 -> 100.2 mm
Other:
- board text added: "I2C"
- board text added: "Open Hardware blood pressure measurement"
- board text added: "VALVE"
- board text added: "uCmini"
- board text added: "wyolum.com"
