File: KiCAD/uCm.kicad_pcb (KiCad board)
At the start: 2 copper layers, 99 x 80 mm, 133 parts, among them J1 5V_EXT, J2 3V3_EXT, P1 AREF, P10 C3SB, P11 VSel_Vlv, P13 PWR_IN, P14 X_VALVE, P17 PUMP, P24 PWR_IN, P34 VSel_Vlv2, P38 X_VALVE2, P4 ICSP, P5 FTDI, P7 GAGE_PR, P9 C3SB, Q1 BCP5416TA, Q2 BCP5416TA, Q3 BCP5416TA, Q4 BCP5416TA, SW1 Reset, SW2 INT0, SW3 INT1, U1 TXB0104D, U2 LM2675-5.0, U3 LM2675-3.3, U5 DS3231N, U7 ATMEGA328-AU-ND, X1 16MHz

Commit message: some mods to PCB layout
Parts:
- added REF**: via01, uCm:via01, F.Cu at (59.7, 84.2)
- added REF**: via01, uCm:via01, F.Cu at (75.8, 76.7)
- added REF**: via01, uCm:via01, F.Cu at (51.6, 76.7)
- added REF**: via01, uCm:via01, F.Cu at (81.6, 80.8)
- added REF**: via01, uCm:via01, F.Cu at (82.8, 81.5)
- added REF**: via01, uCm:via01, F.Cu at (81.4, 89.7)
- added REF**: via01, uCm:via01, F.Cu at (81.4, 88.3)
- added REF**: via01, uCm:via01, F.Cu at (80.1, 89.7)
- added REF**: via01, uCm:via01, F.Cu at (55.8, 80.7)
- added REF**: via01, uCm:via01, F.Cu at (55.8, 82.2)
- added REF**: via01, uCm:via01, F.Cu at (81.6, 82.2)
- added REF**: via01, uCm:via01, F.Cu at (61.1, 84.2)
- added REF**: via01, uCm:via01, F.Cu at (55.6, 88.3)
- added REF**: via01, uCm:via01, F.Cu at (57.1, 81.5)
- added REF**: via01, uCm:via01, F.Cu at (55.6, 89.7)
- added REF**: via01, uCm:via01, F.Cu at (59.7, 80.8)
- added REF**: via01, uCm:via01, F.Cu at (61.1, 80.8)
- added REF**: via01, uCm:via01, F.Cu at (85.5, 84.0)
- added REF**: via01, uCm:via01, F.Cu at (54.3, 89.7)
- added REF**: via01, uCm:via01, F.Cu at (50.1, 76.7)
- added REF**: via01, uCm:via01, F.Cu at (86.8, 84.0)
- added REF**: via01, uCm:via01, F.Cu at (85.5, 80.8)
- added REF**: via01, uCm:via01, F.Cu at (86.8, 80.8)
- added REF**: via01, uCm:via01, F.Cu at (77.2, 76.7)
Routing:
- net GND: track 291.9 -> 320.5 mm
- net /Interface/5V0: track 461.8 -> 463.7 mm
- net /Interface/~PD6_Spk: track 33.5 -> 34.9 mm
- net /Interface/12V: track 278.3 -> 279.4 mm
- added copper zone on F.Cu, net +3.3V
- added copper zone on F.Cu, net /Interface/5V0
- added copper zone on F.Cu, net /pwr/CB3
- added copper zone on F.Cu, net /pwr/CB5
- added copper zone on F.Cu, net /pwr/VSW3
- added copper zone on F.Cu, net /pwr/VSW5
