File: KiCAD/uCm_rtc.sch (KiCad schematic (older format))
At the start: 8 parts, among them U5 DS3231N

Commit message: work in progress
Parts:
- B1, B2, B3: footprint I_O -> uCm:I_O
- BT1: footprint CR2032 -> uCm:CR2032
- C23: footprint c_0805 -> uCm:c_0805
- R11: footprint r_0805 -> uCm:r_0805
- U5: footprint DS3231 -> uCm:DS3231
Changed lines of the file:
@@
 F 0 "U5" H 5850 3350 60  0000 C CNN
 F 1 "DS3231N" H 5250 2400 60  0000 C CNN
-F 2 "DS3231" H 5250 2500 60  0001 C CNN
+F 2 "uCm:DS3231" H 5250 2500 60  0001 C CNN
 F 3 "" H 5550 2800 60  0001 C CNN
 F 4 "IC RTC W/TCXO 16-SOIC" H 5550 3450 60  0001 L CNN "Field4"
@@
 F 0 "R11" H 7050 2150 50  0000 C CNN
 F 1 "10k" V 7155 2000 50  0000 C CNN
-F 2 "r_0805" V 7255 2000 50  0001 C CNN
+F 2 "uCm:r_0805" V 7255 2000 50  0001 C CNN
 F 3 "" H 7150 2000 60  0001 C CNN
 F 4 "RES 10K OHM 1/8W 5% CF AXIAL" H 7150 2100 60  0001 L CNN "Field4"
@@
 F 0 "C23" H 4175 2875 50  0000 L CNN
 F 1 "100nF" V 4250 2450 50  0000 L CNN
-F 2 "c_0805" H 4175 2775 50  0001 C CNN
+F 2 "uCm:c_0805" H 4175 2775 50  0001 C CNN
 F 3 "" H 4175 2775 60  0001 C CNN
 F 4 "CAP FILM 0.1UF 63VDC RADIAL" H 4175 2975 60  0001 L CNN "Field4"
@@
 F 0 "BT1" V 3850 2625 50  0000 L CNN
 F 1 "BATT_HOLDER" H 3975 2675 50  0000 L CNN
-F 2 "CR2032" H 3950 2900 60  0001 L CNN
+F 2 "uCm:CR2032" H 3950 2900 60  0001 L CNN
 F 3 "" H 3950 2800 60  0001 C CNN
 F 4 "HOLDER BATTERY COIN 20MM DIA THM" H 3950 3100 60  0001 L CNN "Field4"
@@
 BAT
 $Comp
-L +BATT #PWR017
+L +BATT #PWR019
 U 1 1 4EC101F0
 P 5300 1850
-F 0 "#PWR017" H 5300 1800 20  0001 C CNN
+F 0 "#PWR019" H 5300 1800 20  0001 C CNN
 F 1 "+BATT" H 5300 1950 30  0000 C CNN
 F 2 "" H 5300 1850 60  0001 C CNN
@@
 F 0 "B3" H 7730 2750 40  0000 L CNN
 F 1 "I_O" H 7650 2805 30  0001 C CNN
-F 2 "I_O" H 7650 2750 60  0001 C CNN
+F 2 "uCm:I_O" H 7650 2750 60  0001 C CNN
 F 3 "" H 7650 2750 60  0001 C CNN
 	1    7650 2750
@@
 F 0 "B2" H 7730 2600 40  0000 L CNN
 F 1 "I_O" H 7650 2655 30  0001 C CNN
-F 2 "I_O" H 7650 2600 60  0001 C CNN
+F 2 "uCm:I_O" H 7650 2600 60  0001 C CNN
 F 3 "" H 7650 2600 60  0001 C CNN
 	1    7650 2600
@@
 F 0 "B1" H 7730 2450 40  0000 L CNN
 F 1 "I_O" H 7650 2505 30  0001 C CNN
-F 2 "I_O" H 7650 2450 60  0001 C CNN
+F 2 "uCm:I_O" H 7650 2450 60  0001 C CNN
 F 3 "" H 7650 2450 60  0001 C CNN
 	1    7650 2450

Commit message: changed power supply section
Parts:
- BT1: Field10 3003K-ND -> (none); Field11 http://www.digikey.com/scripts/DkSearch/dksus.dll?x=0&y=0&l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 -> (none); Field4 HOLDER BATTERY COIN 20MM DIA THM -> (none); Field5 Coin Cell, Retainer -> (none); Field6 Coin, 20.0mm -> (none); Field7 Keystone Electronics -> (none); Field8 3003 -> (none); Field9 Digikey -> (none); manf# (none) -> 3003
- BT2: Field10 P189-ND -> (none); Field11 http://www.digikey.com/product-detail/en/CR2032/P189-ND/319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 -> (none); Field4 BATTERY LITHIUM COIN 3V 20MM -> (none); Field5 Lithium, 3V, 225mAh -> (none); Field6 CR2032 -> (none); Field7 Panasonic - BSG -> (none); Field8 CR2032 -> (none); Field9 Digikey -> (none); manf# (none) -> CR2032
- C23: Field10 399-5863-ND -> (none); Field11 http://www.digikey.com/product-detail/en/R82DC3100AA50J/399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 -> (none); Field4 CAP FILM 0.1UF 63VDC RADIAL -> (none); Field5 100nF, 63V -> (none); Field6 R82 -> (none); Field7 Kemet -> (none); Field8 R82DC3100AA50J -> (none); Field9 Digikey -> (none); manf# (none) -> CL21B104KCC5PNC
- R11: Field10 CF18JT10K0CT-ND -> (none); Field11 http://www.digikey.com/product-detail/en/CF18JT10K0/CF18JT1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 -> (none); Field4 RES 10K OHM 1/8W 5% CF AXIAL -> (none); Field5 0.125W, 1/8W -> (none); Field6 Axial -> (none); Field7 Stackpole Electronics Inc -> (none); Field8 CF18JT10K0 -> (none); Field9 Digikey -> (none); manf# (none) -> RMCF0805JT10K0
- U5: Field10 DS3231S#-ND -> (none); Field11 http://www.digikey.com/product-detail/en/DS3231S%23/DS3231S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 -> (none); Field4 IC RTC W/TCXO 16-SOIC -> (none); Field5 Clock/Calendar -> (none); Field6 16-SOIC (0.295\", 7.50mm Width) -> (none); Field7 Maxim Integrated -> (none); Field8 DS3231S# -> (none); Field9 Digikey -> (none); manf# (none) -> DS3231S#
Changed lines of the file:
@@
 EESchema Schematic File Version 2
 LIBS:uCm
-LIBS:Conn-raspberry
 LIBS:power
 LIBS:uCm-cache
@@
 F 2 "uCm:DS3231" H 5250 2500 60  0001 C CNN
 F 3 "" H 5550 2800 60  0001 C CNN
-F 4 "IC RTC W/TCXO 16-SOIC" H 5550 3450 60  0001 L CNN "Field4"
-F 5 "Clock/Calendar" H 5550 3550 60  0001 L CNN "Field5"
-F 6 "16-SOIC (0.295\", 7.50mm Width)" H 5550 3650 60  0001 L CNN "Field6"
-F 7 "Maxim Integrated" H 5550 3750 60  0001 L CNN "Field7"
-F 8 "DS3231S#" H 5550 3850 60  0001 L CNN "Field8"
-F 9 "Digikey" H 5550 3950 60  0001 L CNN "Field9"
-F 10 "DS3231S#-ND" H 5550 4050 60  0001 L CNN "Field10"
-F 11 "http://www.digikey.com/product-detail/en/DS3231S%23/DS3231S%23-ND/1197574" H 5550 4150 60  0001 L CNN "Field11"
+F 4 "DS3231S#" H 5550 2800 60  0001 C CNN "manf#"
 	1    5550 2800
 	1    0    0    -1
@@
 F 2 "uCm:r_0805" V 7255 2000 50  0001 C CNN
 F 3 "" H 7150 2000 60  0001 C CNN
-F 4 "RES 10K OHM 1/8W 5% CF AXIAL" H 7150 2100 60  0001 L CNN "Field4"
-F 5 "0.125W, 1/8W" H 7150 2200 60  0001 L CNN "Field5"
-F 6 "Axial" H 7150 2300 60  0001 L CNN "Field6"
-F 7 "Stackpole Electronics Inc" H 7150 2400 60  0001 L CNN "Field7"
-F 8 "CF18JT10K0" H 7150 2500 60  0001 L CNN "Field8"
-F 9 "Digikey" H 7150 2600 60  0001 L CNN "Field9"
-F 10 "CF18JT10K0CT-ND" H 7150 2700 60  0001 L CNN "Field10"
-F 11 "http://www.digikey.com/product-detail/en/CF18JT10K0/CF18JT10K0CT-ND/2022766?cur=USD" H 7150 2800 60  0001 L CNN "Field11"
+F 4 "RMCF0805JT10K0" H 7150 2000 60  0001 C CNN "manf#"
 	1    7150 2000
 	1    0    0    -1
@@
 F 2 "uCm:c_0805" H 4175 2775 50  0001 C CNN
 F 3 "" H 4175 2775 60  0001 C CNN
-F 4 "CAP FILM 0.1UF 63VDC RADIAL" H 4175 2975 60  0001 L CNN "Field4"
-F 5 "100nF, 63V" H 4175 3075 60  0001 L CNN "Field5"
-F 6 "R82" H 4175 3175 60  0001 L CNN "Field6"
-F 7 "Kemet" H 4175 3275 60  0001 L CNN "Field7"
-F 8 "R82DC3100AA50J" H 4175 3375 60  0001 L CNN "Field8"
-F 9 "Digikey" H 4175 3475 60  0001 L CNN "Field9"
-F 10 "399-5863-ND" H 4175 3575 60  0001 L CNN "Field10"
-F 11 "http://www.digikey.com/product-detail/en/R82DC3100AA50J/399-5863-ND/2571298?cur=USD" H 4175 3675 60  0001 L CNN "Field11"
+F 4 "CL21B104KCC5PNC" H 4175 2775 60  0001 C CNN "manf#"
 	1    4175 2775
 	1    0    0    -1
@@
 F 2 "" H 3525 2825 60  0001 C CNN
 F 3 "" H 3525 2825 60  0001 C CNN
-F 4 "BATTERY LITHIUM COIN 3V 20MM" H 3525 3125 60  0001 L CNN "Field4"
-F 5 "Lithium, 3V, 225mAh" H 3525 3225 60  0001 L CNN "Field5"
-F 6 "CR2032" H 3525 3325 60  0001 L CNN "Field6"
-F 7 "Panasonic - BSG" H 3525 3425 60  0001 L CNN "Field7"
-F 8 "CR2032" H 3525 3525 60  0001 L CNN "Field8"
-F 9 "Digikey" H 3525 3625 60  0001 L CNN "Field9"
-F 10 "P189-ND" H 3525 3725 60  0001 L CNN "Field10"
-F 11 "http://www.digikey.com/product-detail/en/CR2032/P189-ND/31939?cur=USD" H 3525 3825 60  0001 L CNN "Field11"
+F 4 "CR2032" H 3525 3125 60  0001 L CNN "manf#"
 	1    3525 2825
 	0    1    1    0
@@
 F 2 "uCm:CR2032" H 3950 2900 60  0001 L CNN
 F 3 "" H 3950 2800 60  0001 C CNN
-F 4 "HOLDER BATTERY COIN 20MM DIA THM" H 3950 3100 60  0001 L CNN "Field4"
-F 5 "Coin Cell, Retainer" H 3950 3200 60  0001 L CNN "Field5"
-F 6 "Coin, 20.0mm" H 3950 3300 60  0001 L CNN "Field6"
-F 7 "Keystone Electronics" H 3950 3400 60  0001 L CNN "Field7"
-F 8 "3003" H 3950 3500 60  0001 L CNN "Field8"
-F 9 "Digikey" H 3950 3600 60  0001 L CNN "Field9"
-F 10 "3003K-ND" H 3950 3700 60  0001 L CNN "Field10"
-F 11 "http://www.digikey.com/scripts/DkSearch/dksus.dll?x=0&y=0&lang=en&KeyWords=3003K-ND&cur=USD" H 3950 3800 60  0001 L CNN "Field11"
+F 4 "3003" H 3950 3100 60  0001 L CNN "manf#"
 	1    3950 2800
 	0    1    1    0
@@
 BAT
 $Comp
-L +BATT #PWR020
+L +BATT #PWR019
 U 1 1 4EC101F0
 P 5300 1850
-F 0 "#PWR020" H 5300 1800 20  0001 C CNN
+F 0 "#PWR019" H 5300 1800 20  0001 C CNN
 F 1 "+BATT" H 5300 1950 30  0000 C CNN
 F 2 "" H 5300 1850 60  0001 C CNN
