File: KiCAD/uCm.sch (KiCad schematic (older format))
At the start: 37 parts, among them P1 AREF, P4 ICSP, P5 FTDI, SW1 Reset, SW2 INT0, SW3 INT1, U7 ATMEGA328-AU-ND, X1 16MHz

Commit message: work in progress
Parts:
- removed B13, B14: PB0, I_O, symbol I_O
- B10, B11, B12, B4, B7, B8, B9: footprint I_O -> uCm:I_O
- C1, C28, C4: footprint c_0805 -> uCm:c_0805
- C2, C3: footprint c_0603 -> uCm:c_0603
- P1: footprint ShortLink2 -> uCm:ShortLink2
- P4: footprint Header_ISP -> uCm:Header_ISP
- P5: footprint Header_FTDI -> uCm:Header_FTDI
- R1, R2, R21, R22, R3: footprint r_0805 -> uCm:r_0805
- SC1, SC10, SC2, SC3, SC4, SC5, SC6, SC7, SC8, SC9: footprint vite_3mm -> uCm:vite_3mm
- SW1, SW2, SW3: footprint SW_PB_V_H -> uCm:SW_PB_V_H
- U7: footprint TQFP32 -> uCm:TQFP32
- X1: footprint Xtal_SMD3 -> uCm:Xtal_SMD3
Connections:
- net PD4 renamed PD4_Valve
- net ~PD6 renamed ~PD6_Spk
Other:
- note added: "NOTE\nFTDI is un-powered.\nExternal 5V is required"
- note added: "Speaker PWM"
- note added: "Valve #2"
Changed lines of the file:
@@
 F 0 "P4" V 7425 6175 60  0000 C CNN
 F 1 "ICSP" V 7525 6175 60  0000 C CNN
-F 2 "Header_ISP" V 7625 6175 60  0001 C CNN
+F 2 "uCm:Header_ISP" V 7625 6175 60  0001 C CNN
 F 3 "" H 7475 6175 60  0001 C CNN
 F 4 "CONN HEADER 6POS .100 STR 15AU" H 7475 6275 60  0001 L CNN "Field4"
@@
 F 0 "P1" V 925 1325 50  0000 C CNN
 F 1 "AREF" V 1025 1325 50  0000 C CNN
-F 2 "ShortLink2" V 1125 1325 50  0001 C CNN
+F 2 "uCm:ShortLink2" V 1125 1325 50  0001 C CNN
 F 3 "" H 975 1325 60  0001 C CNN
 F 4 "CONN HEADER 50POS .100\" SGL GOLD" H 975 1425 60  0001 L CNN "Field4"
@@
 F 0 "SW1" V 1650 4550 50  0000 C CNN
 F 1 "Reset" V 1575 4575 50  0000 C CNN
-F 2 "SW_PB_V_H" V 1675 4575 50  0001 C CNN
+F 2 "uCm:SW_PB_V_H" V 1675 4575 50  0001 C CNN
 F 3 "" H 1575 4350 60  0001 C CNN
 F 4 "SWITCH TACTILE SPST-NO 0.05A 12V" H 1575 4560 60  0001 L CNN "Field4"
@@
 F 0 "X1" V 1325 2875 40  0000 C CNN
 F 1 "16MHz" V 1550 2900 40  0000 C CNN
-F 2 "Xtal_SMD3" H 1300 3100 60  0001 C CNN
+F 2 "uCm:Xtal_SMD3" H 1300 3100 60  0001 C CNN
 F 3 "" H 1400 3050 60  0001 C CNN
 F 4 "CER RESONATOR 16.00MHZ" H 1400 3300 60  0001 L CNN "Field4"
@@
 F 0 "R3" H 4750 1600 50  0000 C CNN
 F 1 "10k" V 4805 1450 50  0000 C CNN
-F 2 "r_0805" V 4905 1450 50  0001 C CNN
+F 2 "uCm:r_0805" V 4905 1450 50  0001 C CNN
 F 3 "" H 4800 1450 60  0001 C CNN
 F 4 "RES 10K OHM 1/8W 5% CF AXIAL" H 4800 1550 60  0001 L CNN "Field4"
@@
 F 0 "R2" H 4550 1600 50  0000 C CNN
 F 1 "10k" V 4605 1450 50  0000 C CNN
-F 2 "r_0805" V 4705 1450 50  0001 C CNN
+F 2 "uCm:r_0805" V 4705 1450 50  0001 C CNN
 F 3 "" H 4600 1450 60  0001 C CNN
 F 4 "RES 10K OHM 1/8W 5% CF AXIAL" H 4600 1550 60  0001 L CNN "Field4"
@@
 F 0 "R1" H 1525 1600 50  0000 C CNN
 F 1 "10k" V 1580 1450 50  0000 C CNN
-F 2 "r_0805" V 1680 1450 50  0001 C CNN
+F 2 "uCm:r_0805" V 1680 1450 50  0001 C CNN
 F 3 "" H 1575 1450 60  0001 C CNN
 F 4 "RES 10K OHM 1/8W 5% CF AXIAL" H 1575 1550 60  0001 L CNN "Field4"
@@
 F 0 "C3" V 1125 3125 50  0000 L CNN
 F 1 "22pF" V 1025 3075 50  0000 L CNN
-F 2 "c_0603" V 1125 3350 50  0001 C CNN
+F 2 "uCm:c_0603" V 1125 3350 50  0001 C CNN
 F 3 "" H 1075 3300 60  0001 C CNN
 F 4 "CAP CER 22PF 50V 5% RADIAL" H 1075 3500 60  0001 L CNN "Field4"
@@
 F 0 "C2" V 1125 2625 50  0000 L CNN
 F 1 "22pF" V 1025 2575 50  0000 L CNN
-F 2 "c_0603" V 1125 2850 50  0001 C CNN
+F 2 "uCm:c_0603" V 1125 2850 50  0001 C CNN
 F 3 "" H 1075 2800 60  0001 C CNN
 F 4 "CAP CER 22PF 50V 5% RADIAL" H 1075 3000 60  0001 L CNN "Field4"
@@
 F 0 "C4" H 8850 5550 50  0000 L CNN
 F 1 "100nF" V 8875 5150 50  0000 L CNN
-F 2 "c_0805" H 8950 5475 50  0001 C CNN
+F 2 "uCm:c_0805" H 8950 5475 50  0001 C CNN
 F 3 "" H 8950 5475 60  0001 C CNN
 F 4 "CAP FILM 0.1UF 63VDC RADIAL" H 8950 5675 60  0001 L CNN "Field4"
@@
 F 0 "C1" H 1800 1550 50  0000 L CNN
 F 1 "100nF" H 1800 1350 50  0000 L CNN
-F 2 "c_0805" H 1800 1450 50  0001 C CNN
+F 2 "uCm:c_0805" H 1800 1450 50  0001 C CNN
 F 3 "" H 1800 1450 60  0001 C CNN
 F 4 "CAP FILM 0.1UF 63VDC RADIAL" H 1800 1650 60  0001 L CNN "Field4"
@@
 F 0 "SC1" H 5125 6375 40  0000 C CNN
 F 1 "SCREW" H 5125 6575 40  0001 C CNN
-F 2 "vite_3mm" H 5125 6675 40  0001 C CNN
+F 2 "uCm:vite_3mm" H 5125 6675 40  0001 C CNN
 F 3 "" H 5125 6475 60  0001 C CNN
 	1    5125 6475
@@
 F11 "3V3" B L 10050 1925 40
 F12 "~PB1_Pump" I L 10050 3125 40
+F13 "PD4_Valve2" I L 10050 2625 40
+F14 "~PD6_Spk" I L 10050 2825 40
 $EndSheet
 NoConn ~ 8650 5825
@@
 Blank
 Text Notes 4550 3750 0    40   ~ 0
-Blank
+Speaker PWM
 Text Notes 4550 3650 0    40   ~ 0
 Valve #1 PWM
 Text Notes 4550 3550 0    40   ~ 0
-Blank
+Valve #2
 Text Notes 4550 3350 0    40   ~ 0
 SW INT0
@@
 F 0 "P5" V 8650 6175 60  0000 C CNN
 F 1 "FTDI" V 8750 6175 60  0000 C CNN
-F 2 "Header_FTDI" H 8700 6175 60  0001 C CNN
+F 2 "uCm:Header_FTDI" H 8700 6175 60  0001 C CNN
 F 3 "" H 8700 6175 60  0001 C CNN
 	1    8700 6175
@@
 ~PD5_Valve
 Text Label 4125 3750 0    40   ~ 0
-~PD6
+~PD6_Spk
 Text Label 4125 3450 0    40   ~ 0
 ~PD3
@@
 PD7
 Text Label 4125 3550 0    40   ~ 0
-PD4
+PD4_Valve
 Text Label 4800 650  0    40   ~ 0
 5V0
@@
 F 0 "U7" H 2300 2650 50  0000 L BNN
 F 1 "ATMEGA328-AU-ND" H 2300 2500 50  0000 L BNN
-F 2 "TQFP32" H 3425 1675 50  0001 C CNN
+F 2 "uCm:TQFP32" H 3425 1675 50  0001 C CNN
 F 3 "" H 2900 3250 60  0000 C CNN
 	1    2900 3250
@@
 F 0 "B8" H 4355 2250 40  0000 L CNN
 F 1 "PC0" H 4275 2305 30  0001 C CNN
-F 2 "I_O" H 4275 2250 60  0001 C CNN
+F 2 "uCm:I_O" H 4275 2250 60  0001 C CNN
 F 3 "" H 4275 2250 60  0000 C CNN
 	1    4275 2250
@@
 F 0 "B9" H 4355 2350 40  0000 L CNN
 F 1 "PC1" H 4275 2405 30  0001 C CNN
-F 2 "I_O" H 4275 2350 60  0001 C CNN
+F 2 "uCm:I_O" H 4275 2350 60  0001 C CNN
 F 3 "" H 4275 2350 60  0000 C CNN
 	1    4275 2350
@@
 F 0 "B10" H 4355 2850 40  0000 L CNN
 F 1 "PC6" H 4275 2905 30  0001 C CNN
-F 2 "I_O" H 4275 2850 60  0001 C CNN
+F 2 "uCm:I_O" H 4275 2850 60  0001 C CNN
 F 3 "" H 4275 2850 60  0000 C CNN
 	1    4275 2850
@@
 F 0 "B11" H 4355 2950 40  0000 L CNN
 F 1 "PC7" H 4275 3005 30  0001 C CNN
-F 2 "I_O" H 4275 2950 60  0001 C CNN
+F 2 "uCm:I_O" H 4275 2950 60  0001 C CNN
 F 3 "" H 4275 2950 60  0000 C CNN
 	1    4275 2950
@@
 F 0 "B12" H 4355 4050 40  0000 L CNN
 F 1 "PB0" H 4275 4105 30  0001 C CNN
-F 2 "I_O" H 4275 4050 60  0001 C CNN
+F 2 "uCm:I_O" H 4275 4050 60  0001 C CNN
 F 3 "" H 4275 4050 60  0000 C CNN
 	1    4275 4050
@@
 F 0 "SW2" H 6050 2800 40  0000 C CNN
 F 1 "INT0" H 5550 2800 40  0000 C CNN
-F 2 "SW_PB_V_H" H 5800 2750 60  0001 C CNN
+F 2 "uCm:SW_PB_V_H" H 5800 2750 60  0001 C CNN
 F 3 "" H 5800 2750 60  0000 C CNN
 F 4 "SWITCH TACTILE SPST-NO 0.05A 12V" H 5800 2960 60  0001 L CNN "Field4"
@@
 F 0 "SW3" H 6250 2800 40  0000 C CNN
 F 1 "INT1" H 5750 2800 40  0000 C CNN
-F 2 "SW_PB_V_H" H 6000 2750 60  0001 C CNN
+F 2 "uCm:SW_PB_V_H" H 6000 2750 60  0001 C CNN
 F 3 "" H 6000 2750 60  0000 C CNN
 F 4 "SWITCH TACTILE SPST-NO 0.05A 12V" H 6000 2960 60  0001 L CNN "Field4"
@@
 F 0 "R22" H 5925 4050 50  0000 C CNN
 F 1 "10k" V 6005 3900 50  0000 C CNN
-F 2 "r_0805" V 6105 3900 50  0001 C CNN
+F 2 "uCm:r_0805" V 6105 3900 50  0001 C CNN
 F 3 "" H 6000 3900 60  0001 C CNN
 F 4 "RES 10K OHM 1/8W 5% CF AXIAL" H 6000 4000 60  0001 L CNN "Field4"
@@
 F 0 "R21" H 5725 4050 50  0000 C CNN
 F 1 "10k" V 5805 3900 50  0000 C CNN
-F 2 "r_0805" V 5905 3900 50  0001 C CNN
+F 2 "uCm:r_0805" V 5905 3900 50  0001 C CNN
 F 3 "" H 5800 3900 60  0001 C CNN
 F 4 "RES 10K OHM 1/8W 5% CF AXIAL" H 5800 4000 60  0001 L CNN "Field4"
@@
 F 0 "C28" H 3250 1550 50  0000 L CNN
 F 1 "100nF" H 3250 1350 50  0000 L CNN
-F 2 "c_0805" H 3250 1450 50  0001 C CNN
+F 2 "uCm:c_0805" H 3250 1450 50  0001 C CNN
 F 3 "" H 3250 1450 60  0001 C CNN
 F 4 "CAP FILM 0.1UF 63VDC RADIAL" H 3250 1650 60  0001 L CNN "Field4"
@@
 F 0 "B4" H 4355 3850 40  0000 L CNN
 F 1 "PB0" H 4275 3905 30  0001 C CNN
-F 2 "I_O" H 4275 3850 60  0001 C CNN
+F 2 "uCm:I_O" H 4275 3850 60  0001 C CNN
 F 3 "" H 4275 3850 60  0000 C CNN
 	1    4275 3850
@@
 F 0 "SC3" H 5125 6575 40  0000 C CNN
 F 1 "SCREW" H 5125 6775 40  0001 C CNN
-F 2 "vite_3mm" H 5125 6875 40  0001 C CNN
+F 2 "uCm:vite_3mm" H 5125 6875 40  0001 C CNN
 F 3 "" H 5125 6675 60  0001 C CNN
 	1    5125 6675
@@
 F 0 "SC5" H 5125 6775 40  0000 C CNN
 F 1 "SCREW" H 5125 6975 40  0001 C CNN
-F 2 "vite_3mm" H 5125 7075 40  0001 C CNN
+F 2 "uCm:vite_3mm" H 5125 7075 40  0001 C CNN
 F 3 "" H 5125 6875 60  0001 C CNN
 	1    5125 6875
@@
 F 0 "SC8" H 5125 6975 40  0000 C CNN
 F 1 "SCREW" H 5125 7175 40  0001 C CNN
-F 2 "vite_3mm" H 5125 7275 40  0001 C CNN
+F 2 "uCm:vite_3mm" H 5125 7275 40  0001 C CNN
 F 3 "" H 5125 7075 60  0001 C CNN
 	1    5125 7075
@@
 F 0 "SC6" H 5325 6775 40  0000 C CNN
 F 1 "SCREW" H 5325 6975 40  0001 C CNN
-F 2 "vite_3mm" H 5325 7075 40  0001 C CNN
+F 2 "uCm:vite_3mm" H 5325 7075 40  0001 C CNN
 F 3 "" H 5325 6875 60  0001 C CNN
 	1    5325 6875
@@
 F 0 "SC9" H 5325 6975 40  0000 C CNN
 F 1 "SCREW" H 5325 7175 40  0001 C CNN
-F 2 "vite_3mm" H 5325 7275 40  0001 C CNN
+F 2 "uCm:vite_3mm" H 5325 7275 40  0001 C CNN
 F 3 "" H 5325 7075 60  0001 C CNN
 	1    5325 7075
@@
 F 0 "SC2" H 5525 6375 40  0000 C CNN
 F 1 "SCREW" H 5525 6575 40  0001 C CNN
-F 2 "vite_3mm" H 5525 6675 40  0001 C CNN
+F 2 "uCm:vite_3mm" H 5525 6675 40  0001 C CNN
 F 3 "" H 5525 6475 60  0001 C CNN
 	1    5525 6475
@@
 F 0 "SC4" H 5525 6575 40  0000 C CNN
 F 1 "SCREW" H 5525 6775 40  0001 C CNN
-F 2 "vite_3mm" H 5525 6875 40  0001 C CNN
+F 2 "uCm:vite_3mm" H 5525 6875 40  0001 C CNN
 F 3 "" H 5525 6675 60  0001 C CNN
 	1    5525 6675
@@
 F 0 "SC7" H 5525 6775 40  0000 C CNN
 F 1 "SCREW" H 5525 6975 40  0001 C CNN
-F 2 "vite_3mm" H 5525 7075 40  0001 C CNN
+F 2 "uCm:vite_3mm" H 5525 7075 40  0001 C CNN
 F 3 "" H 5525 6875 60  0001 C CNN
 	1    5525 6875
@@
 F 0 "SC10" H 5525 6975 40  0000 C CNN
 F 1 "SCREW" H 5525 7175 40  0001 C CNN
-F 2 "vite_3mm" H 5525 7275 40  0001 C CNN
+F 2 "uCm:vite_3mm" H 5525 7275 40  0001 C CNN
 F 3 "" H 5525 7075 60  0001 C CNN
 	1    5525 7075
@@
 F 0 "B7" H 4355 2450 40  0000 L CNN
 F 1 "PC1" H 4275 2505 30  0001 C CNN
-F 2 "I_O" H 4275 2450 60  0001 C CNN
+F 2 "uCm:I_O" H 4275 2450 60  0001 C CNN
 F 3 "" H 4275 2450 60  0000 C CNN
 	1    4275 2450
 	1    0    0    -1
 $EndComp
-$Comp
-L I_O B13
-U 1 1 55A3A7AC
-P 4275 3550
-F 0 "B13" H 4355 3550 40  0000 L CNN
-F 1 "PB0" H 4275 3605 30  0001 C CNN
-F 2 "I_O" H 4275 3550 60  0001 C CNN
-F 3 "" H 4275 3550 60  0000 C CNN
-	1    4275 3550
-	1    0    0    -1
-$EndComp
-$Comp
-L I_O B14
-U 1 1 55A3B103
-P 4275 3750
-F 0 "B14" H 4355 3750 40  0000 L CNN
-F 1 "PB0" H 4275 3805 30  0001 C CNN
-F 2 "I_O" H 4275 3750 60  0001 C CNN
-F 3 "" H 4275 3750 60  0000 C CNN
-	1    4275 3750
-	1    0    0    -1
-$EndComp
+Text Notes 8225 6525 0    50   ~ 0
+NOTE\nFTDI is un-powered.\nExternal 5V is required
+Wire Wire Line
+	10050 2625 9600 2625
+Text Label 9600 2625 0    40   ~ 0
+PD4_Valve
+Wire Wire Line
+	10050 2825 9600 2825
+Text Label 9600 2825 0    40   ~ 0
+~PD6_Spk
 $EndSCHEMATC

Commit message: layout, work in progress
Parts:
- removed SC1, SC2, SC3, SC4, SC5, SC8: SCREW, uCm:vite_3mm, symbol SCREW
Connections:
- net 5V0: no longer C1.1
- net AREF: now also C1.1
Other:
- note added: "Valve #1"
- note added: "Valve #2 PWM"
- note removed: "Valve #1 PWM"
- note removed: "Valve #2"
- moved on the sheet: C1
Changed lines of the file:
@@
 L C C1
 U 1 1 50E2940E
-P 1800 1450
-F 0 "C1" H 1800 1550 50  0000 L CNN
-F 1 "100nF" H 1800 1350 50  0000 L CNN
-F 2 "uCm:c_0805" H 1800 1450 50  0001 C CNN
-F 3 "" H 1800 1450 60  0001 C CNN
-F 4 "CAP FILM 0.1UF 63VDC RADIAL" H 1800 1650 60  0001 L CNN "Field4"
-F 5 "100nF, 63V" H 1800 1750 60  0001 L CNN "Field5"
-F 6 "R82" H 1800 1850 60  0001 L CNN "Field6"
-F 7 "Kemet" H 1800 1950 60  0001 L CNN "Field7"
-F 8 "R82DC3100AA50J" H 1800 2050 60  0001 L CNN "Field8"
-F 9 "Digikey" H 1800 2150 60  0001 L CNN "Field9"
-F 10 "399-5863-ND" H 1800 2250 60  0001 L CNN "Field10"
-F 11 "http://www.digikey.com/product-detail/en/R82DC3100AA50J/399-5863-ND/2571298?cur=USD" H 1800 2350 60  0001 L CNN "Field11"
-	1    1800 1450
+P 1200 2050
+F 0 "C1" H 1200 2150 50  0000 L CNN
+F 1 "100nF" H 1200 1950 50  0000 L CNN
+F 2 "uCm:c_0805" H 1200 2050 50  0001 C CNN
+F 3 "" H 1200 2050 60  0001 C CNN
+F 4 "CAP FILM 0.1UF 63VDC RADIAL" H 1200 2250 60  0001 L CNN "Field4"
+F 5 "100nF, 63V" H 1200 2350 60  0001 L CNN "Field5"
+F 6 "R82" H 1200 2450 60  0001 L CNN "Field6"
+F 7 "Kemet" H 1200 2550 60  0001 L CNN "Field7"
+F 8 "R82DC3100AA50J" H 1200 2650 60  0001 L CNN "Field8"
+F 9 "Digikey" H 1200 2750 60  0001 L CNN "Field9"
+F 10 "399-5863-ND" H 1200 2850 60  0001 L CNN "Field10"
+F 11 "http://www.digikey.com/product-detail/en/R82DC3100AA50J/399-5863-ND/2571298?cur=USD" H 1200 2950 60  0001 L CNN "Field11"
+	1    1200 2050
 	1    0    0    -1
 $EndComp
 Text Notes 4550 3450 0    40   ~ 0
 SW INT1
-$Comp
-L SCREW SC1
-U 1 1 50DADA2B
-P 5125 6475
-F 0 "SC1" H 5125 6375 40  0000 C CNN
-F 1 "SCREW" H 5125 6575 40  0001 C CNN
-F 2 "uCm:vite_3mm" H 5125 6675 40  0001 C CNN
-F 3 "" H 5125 6475 60  0001 C CNN
-	1    5125 6475
-	1    0    0    -1
-$EndComp
 Text Notes 5075 7375 0    40   ~ 0
 Mounting Holes
@@
 F13 "PD4_Valve2" I L 10050 2625 40
 F14 "~PD6_Spk" I L 10050 2825 40
+F15 "SCL" I L 10050 3325 40
+F16 "SDA" I L 10050 3425 40
 $EndSheet
 NoConn ~ 8650 5825
@@
 Speaker PWM
 Text Notes 4550 3650 0    40   ~ 0
-Valve #1 PWM
+Valve #2 PWM
 Text Notes 4550 3550 0    40   ~ 0
-Valve #2
+Valve #1
 Text Notes 4550 3350 0    40   ~ 0
 SW INT0
@@
 	1275 2800 1925 2800
 Wire Wire Line
-	1800 4975 1800 1575
+	1800 4975 1800 2450
 Wire Wire Line
 	8950 5000 8950 5350
@@
 Wire Wire Line
 	4125 4550 3900 4550
-Wire Wire Line
-	1800 800  1800 1325
-Connection ~ 1800 800
 Wire Wire Line
 	1575 4650 1575 4975
@@
 Connection ~ 8450 5700
 Wire Wire Line
-	2000 2450 1800 2450
-Connection ~ 1800 2450
+	1800 2450 2000 2450
 Wire Wire Line
 	1275 3300 1925 3300
@@
 $EndComp
 $Comp
-L SCREW SC3
-U 1 1 52230B6D
-P 5125 6675
-F 0 "SC3" H 5125 6575 40  0000 C CNN
-F 1 "SCREW" H 5125 6775 40  0001 C CNN
-F 2 "uCm:vite_3mm" H 5125 6875 40  0001 C CNN
-F 3 "" H 5125 6675 60  0001 C CNN
-	1    5125 6675
-	1    0    0    -1
-$EndComp
-$Comp
-L SCREW SC5
-U 1 1 52230B73
-P 5125 6875
-F 0 "SC5" H 5125 6775 40  0000 C CNN
-F 1 "SCREW" H 5125 6975 40  0001 C CNN
-F 2 "uCm:vite_3mm" H 5125 7075 40  0001 C CNN
-F 3 "" H 5125 6875 60  0001 C CNN
-	1    5125 6875
-	1    0    0    -1
-$EndComp
-$Comp
-L SCREW SC8
-U 1 1 522315D5
-P 5125 7075
-F 0 "SC8" H 5125 6975 40  0000 C CNN
-F 1 "SCREW" H 5125 7175 40  0001 C CNN
-F 2 "uCm:vite_3mm" H 5125 7275 40  0001 C CNN
-F 3 "" H 5125 7075 60  0001 C CNN
-	1    5125 7075
-	1    0    0    -1
-$EndComp
-$Comp
 L SCREW SC6
 U 1 1 522315DB
@@
 $EndComp
 $Comp
-L SCREW SC2
-U 1 1 522315E7
-P 5525 6475
-F 0 "SC2" H 5525 6375 40  0000 C CNN
-F 1 "SCREW" H 5525 6575 40  0001 C CNN
-F 2 "uCm:vite_3mm" H 5525 6675 40  0001 C CNN
-F 3 "" H 5525 6475 60  0001 C CNN
-	1    5525 6475
-	1    0    0    -1
-$EndComp
-$Comp
-L SCREW SC4
-U 1 1 522315ED
-P 5525 6675
-F 0 "SC4" H 5525 6575 40  0000 C CNN
-F 1 "SCREW" H 5525 6775 40  0001 C CNN
-F 2 "uCm:vite_3mm" H 5525 6875 40  0001 C CNN
-F 3 "" H 5525 6675 60  0001 C CNN
-	1    5525 6675
-	1    0    0    -1
-$EndComp
-$Comp
 L SCREW SC7
 U 1 1 522315F3
@@
 Text Label 9600 2825 0    40   ~ 0
 ~PD6_Spk
+Wire Wire Line
+	10050 3325 9600 3325
+Wire Wire Line
+	10050 3425 9600 3425
+Text Label 9600 3425 0    40   ~ 0
+SDA
+Text Label 9600 3325 0    40   ~ 0
+SCL
+$Comp
+L GND #PWR04
+U 1 1 55E8B5A9
+P 1200 2250
+F 0 "#PWR04" H 1200 2250 30  0001 C CNN
+F 1 "GND" H 1200 2180 30  0001 C CNN
+F 2 "" H 1200 2250 60  0001 C CNN
+F 3 "" H 1200 2250 60  0001 C CNN
+	1    1200 2250
+	1    0    0    -1
+$EndComp
+Wire Wire Line
+	1200 1925 1200 1875
+Wire Wire Line
+	1200 1875 975  1875
+Connection ~ 975  1875
+Wire Wire Line
+	1200 2175 1200 2250
 $EndSCHEMATC
