File: KiCAD/mmM.sch (KiCad schematic (older format))
At the start: 29 parts, among them P1 AREF, P4 ICSP, P5 FTDI, SW1 Reset, SW2 INT0, SW3 INT1, U7 ATMEGA328-AU-ND, X1 16MHz

Commit message: Fresh BOM for mmM
Parts:
- C1, C4: value 100n -> 100nF
- U7: value ATMEGA328-AU-ND -> ATMEGA328P-AU-ND
Changed lines of the file:
@@
 P 2900 3250
 F 0 "U7" H 2300 2650 50  0000 L BNN
-F 1 "ATMEGA328-AU-ND" H 2300 2500 50  0000 L BNN
+F 1 "ATMEGA328P-AU-ND" H 2300 2500 50  0000 L BNN
 F 2 "mmM:TQFP32" H 3425 1675 50  0001 C CNN
 F 3 "" H 2900 3250 60  0000 C CNN
@@
 P 1200 2050
 F 0 "C1" H 1225 2125 40  0000 L CNN
-F 1 "100n" H 1225 1950 40  0000 L CNN
+F 1 "100nF" H 1225 1950 40  0000 L CNN
 F 2 "mmM:c_0805" H 1200 2050 60  0001 C CNN
 F 3 "" H 1200 2050 60  0000 C CNN
@@
 P 8950 5475
 F 0 "C4" H 8975 5550 40  0000 L CNN
-F 1 "100n" H 8975 5375 40  0000 L CNN
+F 1 "100nF" H 8975 5375 40  0000 L CNN
 F 2 "mmM:c_0805" H 8950 5475 60  0001 C CNN
 F 3 "" H 8950 5475 60  0000 C CNN
