File: KiCAD/pwr.sch (KiCad schematic (older format))
At the start: 31 parts, among them J1 5V_EXT, J2 3V3_EXT, P13 PWR_IN, P24 PWR_IN, U2 LM2675-5.0, U3 LM2675-3.3

Commit message: Fresh BOM for mmM
Parts:
- J1, J2: Field10 SAM1031-50-ND -> (none); Field11 http://www.digikey.com/scripts/DkSearch/dksus.dll?WT.z_head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 -> (none); Field4 CONN HEADER 50POS .100\" SGL GOLD -> (none); Field5 Header, Unshrouded, Male pin, -> (none); Field6 0.1\" pitch x 50 nos -> (none); Field7 Samtec Inc -> (none); Field8 TSW-150-07-L-S -> (none); Field9 Digikey -> (none); manf# (none) -> PREC003SAAN-RC
Changed lines of the file:
@@
 F 2 "mmM:Header_3" H 6475 4375 60  0001 C CNN
 F 3 "" H 6475 4375 60  0000 C CNN
-F 4 "CONN HEADER 50POS .100\" SGL GOLD" H 6475 4475 60  0001 L CNN "Field4"
-F 5 "Header, Unshrouded, Male pin," H 6475 4575 60  0001 L CNN "Field5"
-F 6 "0.1\" pitch x 50 nos" H 6475 4675 60  0001 L CNN "Field6"
-F 7 "Samtec Inc" H 6475 4775 60  0001 L CNN "Field7"
-F 8 "TSW-150-07-L-S" H 6475 4875 60  0001 L CNN "Field8"
-F 9 "Digikey" H 6475 4975 60  0001 L CNN "Field9"
-F 10 "SAM1031-50-ND" H 6475 5075 60  0001 L CNN "Field10"
-F 11 "http://www.digikey.com/scripts/DkSearch/dksus.dll?WT.z_header=search_go&lang=en&keywords=SAM1031-50-ND&x=15&y=16&cur=USD" H 6475 5175 60  0001 L CNN "Field11"
+F 4 "PREC003SAAN-RC" V 6475 4375 60  0001 C CNN "manf#"
 	1    6475 4375
 	1    0    0    -1
@@
 F 2 "mmM:Header_3" H 6475 2075 60  0001 C CNN
 F 3 "" H 6475 2075 60  0000 C CNN
-F 4 "CONN HEADER 50POS .100\" SGL GOLD" H 6475 2175 60  0001 L CNN "Field4"
-F 5 "Header, Unshrouded, Male pin," H 6475 2275 60  0001 L CNN "Field5"
-F 6 "0.1\" pitch x 50 nos" H 6475 2375 60  0001 L CNN "Field6"
-F 7 "Samtec Inc" H 6475 2475 60  0001 L CNN "Field7"
-F 8 "TSW-150-07-L-S" H 6475 2575 60  0001 L CNN "Field8"
-F 9 "Digikey" H 6475 2675 60  0001 L CNN "Field9"
-F 10 "SAM1031-50-ND" H 6475 2775 60  0001 L CNN "Field10"
-F 11 "http://www.digikey.com/scripts/DkSearch/dksus.dll?WT.z_header=search_go&lang=en&keywords=SAM1031-50-ND&x=15&y=16&cur=USD" H 6475 2875 60  0001 L CNN "Field11"
+F 4 "PREC003SAAN-RC" V 6475 2075 60  0001 C CNN "manf#"
 	1    6475 2075
 	1    0    0    -1
