File: KiCAD/interface.sch (KiCad schematic (older format))
At the start: 33 parts, among them P10 C3SB, P11 VSel_Vlv, P14 X_VALVE, P17 PUMP, P18 Pump_Cable, P34 VSel_Vlv2, P38 X_VALVE2, P7 GAGE_PR, P9 C3SB, Q1 BCP5416TA, Q2 BCP5416TA, Q3 BCP5416TA, Q4 BCP5416TA, U1 TXB0104D

Commit message: added pull down resistors on microcontroller outputs
Parts:
- added R12, R14, R15, R16: 10k, mmM:r_0805, symbol R
Connections:
- net labels removed: 3V3_PR, P_MISO, P_MOSI, P_SCK, P_SS
- wire segments 134 -> 159
Other:
- note added: "3V_PR"
- note added: "MISO"
- note added: "MOSI"
- note added: "SCK"
- note added: "SS"
- moved on the sheet: C13, C14, C31, D1, D3, D9, P11, P34, P38, Q1, Q3, Q4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

Commit message: mods to board layout
Other:
- note added: "If using HCE...5, \nDNP U1, R4, R7\nand Short U1 pins\n1<>14, 2<>13, 3<>12, \n4<>11, 5<>10"
- note removed: "If using HCE...5, DNP\nU1, R4, R7\nand\nShort U1 pins\n1<>14, 2<>13, 3<>12, \n4<>11, 5<>10"
Changed lines of the file:
@@
 Connection ~ 2425 775
 Text Notes 700  2975 0    47   ~ 0
-If using HCE...5, DNP\nU1, R4, R7\nand\nShort U1 pins\n1<>14, 2<>13, 3<>12, \n4<>11, 5<>10
+If using HCE...5, \nDNP U1, R4, R7\nand Short U1 pins\n1<>14, 2<>13, 3<>12, \n4<>11, 5<>10
 Text Notes 2950 1075 0    40   ~ 0
 MISO

Commit message: PCB optimization
Parts:
- U1: footprint mmM:TXB0104D_null -> mmM:TXB0104D
Other:
- moved on the sheet: C17, C27, C29, Q2, R16, R5
Changed lines of the file:
@@
 	2950 2200 2950 1475
 Wire Wire Line
-	1375 6925 2275 6925
-Wire Wire Line
-	2675 6925 4100 6925
+	1375 6925 3000 6925
+Wire Wire Line
+	3400 6925 4100 6925
 Wire Wire Line
 	5025 800  5525 800
@@
 	1050 975  3325 975
 Wire Wire Line
-	5700 2025 4625 2025
-Wire Wire Line
-	3050 6725 3050 6925
+	4625 2025 5700 2025
+Wire Wire Line
+	3650 6725 3650 6925
 Wire Wire Line
 	5675 1175 5675 1025
@@
 L C_POL_1 C27
 U 1 1 51020D1A
-P 3550 6575
-F 0 "C27" V 3600 6350 50  0000 L CNN
-F 1 "100uF" V 3425 6350 50  0000 L CNN
-F 2 "mmM:C_ELCO_SMD_6x8" H 3150 6550 50  0001 C CNN
-F 3 "" H 3550 6575 60  0001 C CNN
-F 4 "UWT1V101MCL1GS" V 3550 6575 60  0001 C CNN "manf#"
-	1    3550 6575
+P 2325 5950
+F 0 "C27" V 2375 5725 50  0000 L CNN
+F 1 "100uF" V 2200 5725 50  0000 L CNN
+F 2 "mmM:C_ELCO_SMD_6x8" H 1925 5925 50  0001 C CNN
+F 3 "" H 2325 5950 60  0001 C CNN
+F 4 "UWT1V101MCL1GS" V 2325 5950 60  0001 C CNN "manf#"
+	1    2325 5950
 	1    0    0    -1
 $EndComp
@@
 F 0 "U1" H 1900 2500 40  0000 C CNN
 F 1 "TXB0104D" H 1900 2400 40  0000 C CNN
-F 2 "mmM:TXB0104D_null" H 1900 2500 40  0001 C CNN
+F 2 "mmM:TXB0104D" H 1900 2500 40  0001 C CNN
 F 3 "" H 1900 2100 60  0001 C CNN
 F 4 "TXB0104DR" H 1900 2100 60  0001 C CNN "manf#"
@@
 L C C17
 U 1 1 50E29685
-P 3775 6600
-F 0 "C17" H 3775 6700 50  0000 L CNN
-F 1 "100nF" H 3775 6500 50  0000 L CNN
-F 2 "mmM:c_0805" H 3775 6600 50  0001 C CNN
-F 3 "" H 3775 6600 60  0001 C CNN
-F 4 "CL21B104KCC5PNC" H 3775 6600 60  0001 C CNN "manf#"
-	1    3775 6600
+P 2550 5975
+F 0 "C17" H 2550 6075 50  0000 L CNN
+F 1 "100nF" H 2550 5875 50  0000 L CNN
+F 2 "mmM:c_0805" H 2550 5975 50  0001 C CNN
+F 3 "" H 2550 5975 60  0001 C CNN
+F 4 "CL21B104KCC5PNC" H 2550 5975 60  0001 C CNN "manf#"
+	1    2550 5975
 	1    0    0    -1
 $EndComp
@@
 L NPN_TIP112G Q2
 U 1 1 520AA298
-P 2475 6825
-F 0 "Q2" V 2375 6925 50  0000 C CNN
-F 1 "BCP5416TA" V 2375 6500 50  0000 C CNN
-F 2 "mmM:SOT223" H 2665 6825 30  0001 C CNN
-F 3 "" H 2475 6825 60  0001 C CNN
-F 4 "BCP5416TA" V 2475 6825 60  0001 C CNN "manf#"
-	1    2475 6825
+P 3200 6825
+F 0 "Q2" V 3150 6650 50  0000 C CNN
+F 1 "BCP5416TA" H 2900 6900 50  0000 C CNN
+F 2 "mmM:SOT223" H 3390 6825 30  0001 C CNN
+F 3 "" H 3200 6825 60  0001 C CNN
+F 4 "BCP5416TA" V 3200 6825 60  0001 C CNN "manf#"
+	1    3200 6825
 	0    1    1    0
 $EndComp
@@
 	1500 5350 3975 5350
 Wire Wire Line
-	1375 6275 2475 6275
+	1375 6275 3200 6275
 $Comp
 L CONN_2 P18
@@
 L R R5
 U 1 1 5245AF3C
-P 3050 5975
-F 0 "R5" H 3100 6150 50  0000 C CNN
-F 1 "4k7" V 3055 5975 50  0000 C CNN
-F 2 "mmM:r_0805" V 3155 5975 50  0001 C CNN
-F 3 "" H 3050 5975 60  0001 C CNN
-F 4 "RMCF0805JT4K70" H 3050 5975 60  0001 C CNN "manf#"
-	1    3050 5975
+P 3650 5975
+F 0 "R5" H 3700 6150 50  0000 C CNN
+F 1 "4k7" V 3655 5975 50  0000 C CNN
+F 2 "mmM:r_0805" V 3755 5975 50  0001 C CNN
+F 3 "" H 3650 5975 60  0001 C CNN
+F 4 "RMCF0805JT4K70" H 3650 5975 60  0001 C CNN "manf#"
+	1    3650 5975
 	1    0    0    -1
 $EndComp
@@
 L C C29
 U 1 1 5245AF72
-P 3050 6600
-F 0 "C29" H 3075 6675 50  0000 L CNN
-F 1 "100nF" H 3050 6500 50  0000 L CNN
-F 2 "mmM:c_0805" H 3050 6600 50  0001 C CNN
-F 3 "" H 3050 6600 60  0001 C CNN
-F 4 "CL21B104KCC5PNC" H 3050 6600 60  0001 C CNN "manf#"
-	1    3050 6600
-	1    0    0    -1
-$EndComp
-Text Label 3250 6275 0    40   ~ 0
+P 3650 6600
+F 0 "C29" H 3675 6675 50  0000 L CNN
+F 1 "100nF" H 3650 6500 50  0000 L CNN
+F 2 "mmM:c_0805" H 3650 6600 50  0001 C CNN
+F 3 "" H 3650 6600 60  0001 C CNN
+F 4 "CL21B104KCC5PNC" H 3650 6600 60  0001 C CNN "manf#"
+	1    3650 6600
+	1    0    0    -1
+$EndComp
+Text Label 3725 6275 0    40   ~ 0
 Pump
 Wire Wire Line
@@
 	4100 5350 4100 6925
 Wire Wire Line
-	4000 6275 3050 6275
-Wire Wire Line
-	3050 6225 3050 6475
-Wire Wire Line
-	3050 5650 3050 5725
-Wire Wire Line
-	1500 5650 3050 5650
-Connection ~ 3050 6275
-Wire Wire Line
-	3550 6475 3550 5350
-Connection ~ 3550 5350
-Wire Wire Line
-	3775 6475 3775 5350
-Connection ~ 3775 5350
-Wire Wire Line
-	3775 6725 3775 6925
-Connection ~ 3775 6925
-Wire Wire Line
-	3550 6725 3550 6925
-Connection ~ 3550 6925
+	4000 6275 3650 6275
+Wire Wire Line
+	3650 6225 3650 6475
+Wire Wire Line
+	3650 5650 3650 5725
+Wire Wire Line
+	1500 5650 3650 5650
+Connection ~ 3650 6275
 Text Label 1500 5650 0    40   ~ 0
 5V0
@@
 	1375 6975 1375 6925
 Wire Wire Line
-	2475 6275 2475 6625
-Connection ~ 3050 6925
+	3200 6275 3200 6625
+Connection ~ 3650 6925
 Wire Wire Line
 	6025 3275 6650 3275
@@
 	6025 3275 6025 3875
 Wire Wire Line
-	5725 4075 4650 4075
+	4650 4075 5725 4075
 Wire Wire Line
 	5700 3225 5700 3075
@@
 Text HLabel 8900 1200 0    40   Input ~ 0
 SDA
-Text Label 3250 6925 0    40   ~ 0
+Text Label 3725 6925 0    40   ~ 0
 Pump_Ret
 $Comp
@@
 L R R16
 U 1 1 5668192A
-P 1800 6600
-F 0 "R16" H 1875 6775 50  0000 C CNN
-F 1 "10k" V 1805 6600 50  0000 C CNN
-F 2 "mmM:r_0805" V 1905 6600 50  0001 C CNN
-F 3 "" H 1800 6600 60  0001 C CNN
-F 4 "RMCF0805JT10K0" H 1800 6600 60  0001 C CNN "manf#"
-	1    1800 6600
+P 2900 6600
+F 0 "R16" H 2975 6775 50  0000 C CNN
+F 1 "10k" V 2905 6600 50  0000 C CNN
+F 2 "mmM:r_0805" V 3005 6600 50  0001 C CNN
+F 3 "" H 2900 6600 60  0001 C CNN
+F 4 "RMCF0805JT10K0" H 2900 6600 60  0001 C CNN "manf#"
+	1    2900 6600
 	-1   0    0    1
 $EndComp
 Wire Wire Line
-	1800 6350 1800 6275
-Connection ~ 1800 6275
-Wire Wire Line
-	1800 6850 1800 6925
-Connection ~ 1800 6925
+	2900 6350 2900 6275
+Connection ~ 2900 6275
+Wire Wire Line
+	2900 6850 2900 6925
+Connection ~ 2900 6925
 $Comp
 L R R15
@@
 Wire Wire Line
 	4900 4200 4975 4200
+Wire Wire Line
+	2550 5850 2550 5350
+Connection ~ 2550 5350
+Wire Wire Line
+	2325 5850 2325 5350
+Connection ~ 2325 5350
+Wire Wire Line
+	2550 6100 2550 6925
+Connection ~ 2550 6925
+Wire Wire Line
+	2325 6100 2325 6925
+Connection ~ 2325 6925
 $EndSCHEMATC
