File: KiCAD/mmM.kicad_pcb (KiCad board)
At the start: 2 copper layers, 99 x 80 mm, 162 parts, among them J1 5V_EXT, J2 3V3_EXT, P1 AREF, P10 C3SB, P11 VSel_Vlv, P13 PWR_IN, P14 X_VALVE, P17 PUMP, P24 PWR_IN, P34 VSel_Vlv2, P38 X_VALVE2, P4 ICSP, P5 FTDI, P7 GAGE_PR, P9 C3SB, Q1 BCP5416TA, Q2 BCP5416TA, Q3 BCP5416TA, Q4 BCP5416TA, SW1 Reset, SW2 INT0, SW3 INT1, U1 TXB0104D, U2 LM2675-5.0, U3 LM2675-3.3, U5 DS3231N, U7 ATMEGA328P-AU-ND, X1 16MHz

Commit message: PCB optimization
Parts:
- added REF60: via01, uCm:via01, F.Cu at (77.2, 81.7)
- added REF61: via01, uCm:via01, F.Cu at (75.8, 81.7)
- added REF62: via01, uCm:via01, F.Cu at (74.3, 81.7)
- U1: footprint uCm:TXB0104D_null -> mmM:TXB0104D
- moved C27 9.81 mm to (70.0, 27.8), turned to 90 degrees
- moved C17 9.65 mm to (70.0, 23.6), turned to 0 degrees
- moved R16 4.74 mm to (64.3, 40.5), turned to 270 degrees
- moved R5 4.68 mm to (60.0, 40.5)
- moved C29 4.64 mm to (62.1, 40.5)
- moved REF59 1.10 mm to (64.3, 43.8)
- moved REF46 0.90 mm to (69.3, 61.8)
- moved B12 0.61 mm to (67.3, 69.0)
- moved B4 0.50 mm to (66.0, 69.0)
- moved B7 0.40 mm to (71.0, 55.9)
- moved REF26 0.10 mm to (74.3, 76.7)
Connections:
- C17 pad 2: /Interface/Pump_Ret -> GND
- C27 pad 2: /Interface/Pump_Ret -> GND
Routing:
- net GND: track 869.5 -> 890.2 mm
- net /Interface/12V: track 283.5 -> 263.5 mm
- net /Interface/5V0: track 501.2 -> 511.9 mm
- net /Interface/Pump_Ret: track 30.9 -> 22.9 mm
- net /Interface/Pump: track 35.2 -> 28.1 mm
- net /Interface/~PB1_Pump: track 41.4 -> 46.3 mm
- net /Interface/MISO: track 125.3 -> 127.7 mm
- net /Interface/SDA: track 52.4 -> 50.3 mm
- net /~PD3: track 66.4 -> 67.9 mm
- net /PD2: track 78.1 -> 79.4 mm
- net /Interface/PD4_Valve2: track 20.0 -> 18.9 mm
- net /RESET: track 107.5 -> 106.4 mm
- net /Interface/~SS: track 91.3 -> 90.4 mm
- net +3.3V: track 140.9 -> 141.9 mm
- net /Interface/SCL: track 54.5 -> 53.6 mm
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
Commit message: BoM and 3D render work in progress
Parts:
- B1, B10, B11, B12, B2, B3, B4, B7, B8, B9: footprint uCm:I_O -> mmM:I_O
- BT1: footprint uCm:CR2032 -> mmM:CR2032
- C1, C10, C11, C12, C13, C14, C15, C17, C23, C28, C29, C31, C4, C7, C8, C9: footprint uCm:c_0805 -> mmM:c_0805
- C16, C18: footprint uCm:C_2917_HandSoldering -> mmM:C_2917_HandSoldering
- C2, C3: footprint uCm:c_0603 -> mmM:c_0603
- C27: footprint uCm:C_ELCO_SMD -> mmM:C_ELCO_SMD
- C5, C6: footprint uCm:C_ELCO_SMD_8x10 -> mmM:C_ELCO_SMD_8x10
- D1, D3, D4, D9: footprint uCm:diode-DO214AC -> mmM:diode-DO214AC
- D10, D2: footprint uCm:DO-214AB -> mmM:DO-214AB
- D5, D6, D7, D8: footprint uCm:led_0805 -> mmM:led_0805
- G1, G2: footprint uCm:Logo-WL3 -> mmM:Logo-WL3
- G3, G4: footprint uCm:OSHW_6mm -> mmM:OSHW_6mm
- J1, J2, P11, P34: footprint uCm:Header_3 -> mmM:Header_3
- L1, L2: footprint uCm:Choke_SMD_Wuerth-784775133 -> mmM:Choke_SMD_Wuerth-784775133
- P1: footprint uCm:ShortLink2 -> mmM:ShortLink2
- P10, P9: footprint uCm:pin_strip_4-90 -> mmM:pin_strip_4-90
- P13: footprint uCm:Header_2 -> mmM:Header_2
- P14, P38: footprint uCm:X_Valve_2 -> mmM:X_Valve_2
- P17: footprint uCm:Pump_P54E01R_03 -> mmM:Pump_P54E01R_03
- P24: footprint uCm:JACK_ALIM -> mmM:JACK_ALIM
- P4: footprint uCm:Header_ISP -> mmM:Header_ISP
- P5: footprint uCm:Header_FTDI -> mmM:Header_FTDI
- P7: footprint uCm:HCEM500GUH9P3 -> mmM:HCEM500GUH9P3
- Q1, Q2, Q3, Q4: footprint uCm:SOT223 -> mmM:SOT223
- R1, R10, R11, R13, R2, R21, R22, R3, R4, R5, R6, R7, R8, R9, W1, W2: footprint uCm:r_0805 -> mmM:r_0805
- REF1, REF10, REF11, REF12, REF13, REF14, REF15, REF16, REF17, REF18, REF19, REF2, REF20, REF21, REF22, REF23, REF24, REF25, REF26, REF27, REF3, REF4, REF5, REF55, REF56, REF57, REF58, REF6, REF60, REF61, REF62, REF7, REF8, REF9: footprint uCm:via01 -> mmM:via01
- REF28, REF29, REF30, REF31, REF32, REF33, REF34, REF35, REF36, REF37, REF38, REF39, REF40, REF41, REF42, REF43, REF44, REF45, REF46, REF47, REF48, REF49, REF50, REF51, REF52, REF53, REF54, REF59: footprint uCm:via_th -> mmM:via_th
- SC10, SC6, SC7, SC9: footprint uCm:vite_3mm -> mmM:vite_3mm
- SP1: footprint uCm:Speaker -> mmM:Speaker
- SW1, SW2, SW3: footprint uCm:SW_PB_V_H -> mmM:SW_PB_V_H
- U2, U3: footprint uCm:SO8E -> mmM:SO8E
- U5: footprint uCm:DS3231 -> mmM:DS3231
- U7: footprint uCm:TQFP32 -> mmM:TQFP32
- X1: footprint uCm:Xtal_SMD3 -> mmM:Xtal_SMD3

Commit message: 3D render work in progress
Routing:
- net GND: track 890.2 -> 891.9 mm
Changed lines of the file:
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@@
-(kicad_pcb (version 4) (host pcbnew 4.0.0-2.201512072331+6194~38~ubuntu15.04.1-stable)
+(kicad_pcb (version 4) (host pcbnew 4.0.1-2.201512121406+6195~38~ubuntu15.10.1-stable)
   (general
     (links 308)
     (no_connects 0)
-    (area 13.936499 13.936499 113.063501 94.063501)
+    (area 12.823 13.899999 126.418668 101.828801)
     (thickness 1.6)
     (drawings 137)
@@
     (39 F.Mask user)
     (40 Dwgs.User user)
-    (41 Cmts.User user)
-    (42 Eco1.User user)
-    (43 Eco2.User user)
+    (41 Cmts.User user hide)
+    (42 Eco1.User user hide)
+    (43 Eco2.User user hide)
     (44 Edge.Cuts user)
   )
@@
     )
   )
-  (module mmM:C_ELCO_SMD (layer F.Cu)
-    (at 70.05 27.75 90)
-    (attr smd)
-    (fp_text reference C27 (at 0 -5.15 180) (layer F.SilkS)
-      (effects (font (size 0.8 0.8) (thickness 0.12)))
-    )
-    (fp_text value 100uF (at 0 0 90) (layer F.SilkS) hide
-      (effects (font (size 0.8 0.8) (thickness 0.12)))
-    )
-    (fp_text user [+] (at 1.7 3.5 180) (layer F.SilkS)
-      (effects (font (size 0.635 0.635) (thickness 0.127)))
-    )
-    (fp_arc (start 0 0) (end -1.2065 2.3495) (angle 90) (layer F.SilkS) (width 0.1524))
-    (fp_arc (start 0 0) (end -2.3495 1.2065) (angle 90) (layer F.SilkS) (width 0.1524))
-    (fp_line (start -2.667 2.032) (end -2.667 -2.667) (layer F.SilkS) (width 0.1524))
-    (fp_arc (start 0 0) (end 2.3495 -1.143) (angle 90) (layer F.SilkS) (width 0.1524))
-    (fp_arc (start 0.0635 0) (end 1.0795 -2.3495) (angle 90) (layer F.SilkS) (width 0.1524))
-    (fp_line (start 2.667 -2.667) (end 1.016 -2.667) (layer F.SilkS) (width 0.1524))
-    (fp_line (start -2.667 -2.667) (end -1.143 -2.667) (layer F.SilkS) (width 0.1524))
-    (fp_line (start -2.032 2.667) (end -1.0795 2.667) (layer F.SilkS) (width 0.1524))
-    (fp_line (start 2.032 2.667) (end 1.0795 2.667) (layer F.SilkS) (width 0.1524))
-    (fp_line (start 2.032 2.667) (end 2.667 2.032) (layer F.SilkS) (width 0.1524))
-    (fp_line (start 2.667 2.032) (end 2.667 0) (layer F.SilkS) (width 0.1524))
-    (fp_line (start -2.032 2.667) (end -2.667 2.032) (layer F.SilkS) (width 0.1524))
-    (fp_line (start 2.667 -2.667) (end 2.667 0) (layer F.SilkS) (width 0.1524))
-    (pad 1 smd rect (at 0 2.286 90) (size 1.6256 3.048) (layers F.Cu F.Paste F.Mask)
-      (net 7 /Interface/12V))
-    (pad 2 smd rect (at -0.0635 -2.286 90) (size 1.6256 3.048) (layers F.Cu F.Paste F.Mask)
-      (net 32 GND))
-    (model c_elec_5x5_3.wrl
-      (at (xyz 0 0 0))
-      (scale (xyz 1 1 1))
-      (rotate (xyz 0 0 90))
-    )
-  )
   (module mmM:diode-DO214AC (layer F.Cu)
     (at 42.25 48.5 90)
@@
     )
   )
+  (module mmM:C_ELCO_SMD (layer F.Cu)
+    (at 70.05 27.75 90)
+    (attr smd)
+    (fp_text reference C27 (at 0 -5.15 180) (layer F.SilkS)
+      (effects (font (size 0.8 0.8) (thickness 0.12)))
+    )
+    (fp_text value 100uF (at 0 0 90) (layer F.SilkS) hide
+      (effects (font (size 0.8 0.8) (thickness 0.12)))
+    )
+    (fp_text user [+] (at 1.7 3.5 180) (layer F.SilkS)
+      (effects (font (size 0.635 0.635) (thickness 0.127)))
+    )
+    (fp_arc (start 0 0) (end -1.2065 2.3495) (angle 90) (layer F.SilkS) (width 0.1524))
+    (fp_arc (start 0 0) (end -2.3495 1.2065) (angle 90) (layer F.SilkS) (width 0.1524))
+    (fp_line (start -2.667 2.032) (end -2.667 -2.667) (layer F.SilkS) (width 0.1524))
+    (fp_arc (start 0 0) (end 2.3495 -1.143) (angle 90) (layer F.SilkS) (width 0.1524))
+    (fp_arc (start 0.0635 0) (end 1.0795 -2.3495) (angle 90) (layer F.SilkS) (width 0.1524))
+    (fp_line (start 2.667 -2.667) (end 1.016 -2.667) (layer F.SilkS) (width 0.1524))
+    (fp_line (start -2.667 -2.667) (end -1.143 -2.667) (layer F.SilkS) (width 0.1524))
+    (fp_line (start -2.032 2.667) (end -1.0795 2.667) (layer F.SilkS) (width 0.1524))
+    (fp_line (start 2.032 2.667) (end 1.0795 2.667) (layer F.SilkS) (width 0.1524))
+    (fp_line (start 2.032 2.667) (end 2.667 2.032) (layer F.SilkS) (width 0.1524))
+    (fp_line (start 2.667 2.032) (end 2.667 0) (layer F.SilkS) (width 0.1524))
+    (fp_line (start -2.032 2.667) (end -2.667 2.032) (layer F.SilkS) (width 0.1524))
+    (fp_line (start 2.667 -2.667) (end 2.667 0) (layer F.SilkS) (width 0.1524))
+    (pad 1 smd rect (at 0 2.9 90) (size 1.4 3.8) (layers F.Cu F.Paste F.Mask)
+      (net 7 /Interface/12V))
+    (pad 2 smd rect (at 0 -2.85 90) (size 1.4 3.8) (layers F.Cu F.Paste F.Mask)
+      (net 32 GND))
+    (model c_elec_5x5_3.wrl
+      (at (xyz 0 0 0))
+      (scale (xyz 1 1 1))
+      (rotate (xyz 0 0 90))
+    )
+  )
   (gr_line (start 39.25 73.5) (end 35.25 73.5) (angle 90) (layer F.SilkS) (width 0.2))
   (gr_line (start 79.5 73.5) (end 90 73.5) (angle 90) (layer F.SilkS) (width 0.2))
@@
   (segment (start 38.81 62) (end 39.54 61.27) (width 0.762) (layer F.Cu) (net 6) (status 20))
   (segment (start 52.175 60) (end 45.825 60) (width 0.762) (layer F.Cu) (net 6) (status 30))
+  (segment (start 76.2 27.75) (end 72.95 27.75) (width 0.762) (layer F.Cu) (net 7))
+  (segment (start 72.95 24.313) (end 72.95 27.75) (width 0.762) (layer F.Cu) (net 7))
+  (segment (start 70.85 23.55) (end 72.187 23.55) (width 0.762) (layer F.Cu) (net 7))
+  (segment (start 72.187 23.55) (end 72.95 24.313) (width 0.762) (layer F.Cu) (net 7))
   (segment (start 58.25 51.4) (end 58.25 47.4) (width 0.762) (layer B.Cu) (net 7))
   (segment (start 58.25 47.4) (end 56.81 45.96) (width 0.762) (layer B.Cu) (net 7))
-  (segment (start 72.336 27.75) (end 76.2 27.75) (width 0.762) (layer F.Cu) (net 7) (status 10))
   (segment (start 79.5 31.05) (end 79.5 33.5) (width 0.762) (layer F.Cu) (net 7))
   (segment (start 76.2 27.75) (end 79.5 31.05) (width 0.762) (layer F.Cu) (net 7))
-  (segment (start 70.85 23.55) (end 70.85 24.95) (width 0.762) (layer F.Cu) (net 7) (status 10))
-  (segment (start 72.336 26.436) (end 72.336 27.75) (width 0.762) (layer F.Cu) (net 7) (status 20))
-  (segment (start 70.85 24.95) (end 72.336 26.436) (width 0.762) (layer F.Cu) (net 7))
   (segment (start 77.9 43.7) (end 74.4 43.7) (width 0.762) (layer F.Cu) (net 7))
   (segment (start 56 44.8) (end 56 45.96) (width 0.762) (layer F.Cu) (net 7) (status 20))
@@
   (segment (start 102.25 41.5) (end 102.25 40.65) (width 0.254) (layer F.Cu) (net 31) (status 20))
   (segment (start 102.25 40.65) (end 102.25 41) (width 0.254) (layer F.Cu) (net 31) (status 30))
+  (segment (start 72.5 33.7) (end 72.5 31.9) (width 0.762) (layer F.Cu) (net 32))
+  (segment (start 72.5 31.9) (end 71.25 30.65) (width 0.762) (layer F.Cu) (net 32))
+  (segment (start 68.45 30.65) (end 67.2 29.4) (width 0.762) (layer F.Cu) (net 32))
+  (segment (start 71.25 30.65) (end 68.45 30.65) (width 0.762) (layer F.Cu) (net 32))
+  (segment (start 67.2 29.4) (end 67.2 27.75) (width 0.762) (layer F.Cu) (net 32))
+  (segment (start 69.05 23.55) (end 67.713 23.55) (width 0.762) (layer F.Cu) (net 32))
+  (segment (start 67.713 23.55) (end 67.2 24.063) (width 0.762) (layer F.Cu) (net 32))
+  (segment (start 67.2 24.063) (end 67.2 27.75) (width 0.762) (layer F.Cu) (net 32))
   (segment (start 48.7 76.7) (end 46.8 76.7) (width 0.762) (layer F.Cu) (net 32))
   (segment (start 46.8 76.7) (end 44.5 74.4) (width 0.762) (layer F.Cu) (net 32))
@@
   (segment (start 60.75 87.95) (end 60.75 86.46) (width 0.762) (layer F.Cu) (net 32) (status 20))
   (segment (start 60.4 88.3) (end 60.75 87.95) (width 0.762) (layer F.Cu) (net 32))
-  (segment (start 72.5 33.7) (end 72.5 31.9) (width 0.762) (layer F.Cu) (net 32) (status 10))
-  (segment (start 67.764 29.264) (end 67.764 27.8135) (width 0.762) (layer F.Cu) (net 32) (status 20))
-  (segment (start 69.15 30.65) (end 67.764 29.264) (width 0.762) (layer F.Cu) (net 32))
-  (segment (start 71.25 30.65) (end 69.15 30.65) (width 0.762) (layer F.Cu) (net 32))
-  (segment (start 72.5 31.9) (end 71.25 30.65) (width 0.762) (layer F.Cu) (net 32))
-  (segment (start 69.05 23.55) (end 69.05 25) (width 0.762) (layer F.Cu) (net 32) (status 10))
-  (segment (start 69.05 25) (end 67.764 26.286) (width 0.762) (layer F.Cu) (net 32))
-  (segment (start 67.764 26.286) (end 67.764 27.8135) (width 0.762) (layer F.Cu) (net 32) (status 20))
   (segment (start 64.35 41.45) (end 64.35 43.8) (width 0.762) (layer F.Cu) (net 32) (status 30))
   (segment (start 64.35 43.8) (end 59.2 43.8) (width 0.762) (layer B.Cu) (net 32) (status 10))
