File: kicad/mmM.kicad_pcb (KiCad board)
At the start: 2 copper layers, 99 x 80 mm, 165 parts, among them J1 5V_EXT, J2 3V3_EXT, P1 AREF, P10 C3SB, P11 VSel_Vlv, P13 PWR_IN, P14 X_VALVE, P17 PUMP, P24 PWR_IN, P34 VSel_Vlv2, P38 X_VALVE2, P4 ICSP, P5 FTDI, P7 GAGE_PR, P9 C3SB, Q1 BCP5416TA, Q2 BCP5416TA, Q3 BCP5416TA, Q4 BCP5416TA, SW1 Reset, SW2 INT0, SW3 INT1, U1 TXB0104D, U2 LM2675-5.0, U3 LM2675-3.3, U5 DS3231N, U7 ATMEGA328P-AU-ND, X1 16MHz

Commit message: added Cap across RST sw. Fresh Gerbers, PDF. Final v1 ready for prototype
Parts:
- added C19: 100nF, mmM:c_0805, F.Cu at (98.0, 93.5)
- added G3: Logo_OH, mmM:OSHW_6mm, F.Cu at (278.5, 170.5)
- moved REF15 54.6 mm to (117.4, 129.3)
- moved B1 54.6 mm to (120.7, 93.2)
- moved B10 54.6 mm to (109.7, 104.4)
- moved B11 54.6 mm to (109.7, 102.0)
- moved B12 54.6 mm to (103.3, 110.0)
- moved B2 54.6 mm to (120.7, 91.3)
- moved B3 54.6 mm to (120.7, 95.7)
- moved B4 54.6 mm to (102.0, 110.0)
- moved B7 54.6 mm to (107.0, 96.9)
- moved B8 54.6 mm to (109.7, 100.3)
- moved B9 54.6 mm to (109.7, 98.7)
- moved BT1 54.6 mm to (136.8, 96.5)
- moved C1 54.6 mm to (115.7, 103.5)
- moved C10 54.6 mm to (70.0, 66.0)
- moved C11 54.6 mm to (118.8, 81.5)
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Connections:
- P17 pad 3: (no net) -> Net-(P17-Pad3)
- P17 pad 5: (no net) -> Net-(P17-Pad5)
- P5 pad 3: (no net) -> Net-(P5-Pad3)
- P7 pad 7: (no net) -> Net-(P7-Pad7)
- U1 pad 6: (no net) -> Net-(U1-Pad6)
- U1 pad 9: (no net) -> Net-(U1-Pad9)
Routing:
- net /RESET: track 106.4 -> 110.5 mm
- net /PD2: track 79.4 -> 81.3 mm
- net GND: track 892.2 -> 893.6 mm
- net /~PD3: track 67.9 -> 68.7 mm
Other:
- board text added: "This documentation describes Open Hardware and is licensed under the CERN OHL v. 1.2. You may redistribute and modify this documentation under the terms of the CERN OHL v.1.2. (http://ohwr.org/cernohl). This documentation is distributed WITHOUT ANY EXPRESS OR IMPLIED WARRANTY, INCLUDING OF MERCHANTABILITY, SATISFACTORY QUALITY AND FITNESS FOR A PARTICULAR PURPOSE. Please see the CERN OHL v.1.2 fo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"
