File: kicad/mmM.kicad_pcb (KiCad board)
At the start: 2 copper layers, 99 x 80 mm, 167 parts, among them J1 5V_EXT, J2 3V3_EXT, P1 AREF, P10 C3SB, P11 VSel_Vlv, P13 PWR_IN, P14 X_VALVE, P17 PUMP, P24 PWR_IN, P34 VSel_Vlv2, P38 X_VALVE2, P4 ICSP, P5 FTDI, P7 GAGE_PR, P9 C3SB, Q1 BCP5416TA, Q2 BCP5416TA, Q3 BCP5416TA, Q4 BCP5416TA, SW1 Reset, SW2 INT0, SW3 INT1, U1 TXB0104D, U2 LM2675-5.0, U3 LM2675-3.3, U5 DS3231N, U7 ATMEGA328P-AU-ND, X1 16MHz

Commit message: bard convert to ver 10
Connections:
- net /Interface/~MOSI renamed /Interface/~{MOSI}
- net /Interface/~PB1_Pump renamed /Interface/~{PB1_Pump}
- net /Interface/~PD5_Valve renamed /Interface/~{PD5_Valve}
- net /Interface/~PD6_Spk renamed /Interface/~{PD6_Spk}
- net /Interface/~SS renamed /Interface/~{SS}
- net /~PD3 renamed /~{PD3}
- net /~RTS renamed /~{RTS}
Other:
- net class 10mil_PSU removed
- net class 15mil removed
- net class 20mil removed
- net class 25mil removed
- net class 30mil removed
- net class Default removed
