File: kicad/pwr.sch (KiCad schematic (older format))
At the start: 31 parts, among them J1 5V_EXT, J2 3V3_EXT, P13 PWR_IN, P24 PWR_IN, U2 LM2675-5.0, U3 LM2675-3.3

Commit message: made a pretty schematic, fresh symbols
Other:
- note added: "3V3 Regulator"
- note added: "5V0 Regulator"
- note removed: "3V3 Regulator for uControl"
- note removed: "5V0 Regulator for uControl"
