File: kicad/rtc.sch (KiCad schematic (older format))
At the start: 8 parts, among them U5 DS3231N

Commit message: made a pretty schematic, fresh symbols
Changed lines of the file:
@@
 encoding utf-8
 Sheet 4 4
-Title "mmMercury - Open Source Blood Pressure Measurement Platform"
+Title "mmMercury : Blood Pressure Measurement Platform"
 Date "2015-12-27"
 Rev "1"
@@
 U 1 1 50E2C1B1
 P 5550 2800
-F 0 "U5" H 5850 3350 60  0000 C CNN
-F 1 "DS3231N" H 5250 2400 60  0000 C CNN
-F 2 "mmM:DS3231" H 5250 2500 60  0001 C CNN
-F 3 "" H 5550 2800 60  0001 C CNN
-F 4 "DS3231S#" H 5550 2800 60  0001 C CNN "manf#"
+F 0 "U5" H 5450 3350 40  0000 C CNB
+F 1 "DS3231N" H 5550 3450 40  0000 C CNB
+F 2 "mmM:DS3231" H 5250 2500 40  0001 C CNN
+F 3 "" H 5550 2800 40  0001 C CNN
+F 4 "DS3231S#" H 5550 2800 40  0001 C CNN "manf#"
 	1    5550 2800
 	1    0    0    -1
@@
 U 1 1 50E2B876
 P 7150 2000
-F 0 "R11" H 7050 2150 50  0000 C CNN
-F 1 "10k" V 7155 2000 50  0000 C CNN
-F 2 "mmM:r_0805" V 7255 2000 50  0001 C CNN
-F 3 "" H 7150 2000 60  0001 C CNN
-F 4 "RMCF0805JT10K0" H 7150 2000 60  0001 C CNN "manf#"
+F 0 "R11" H 7225 2175 40  0000 C CNB
+F 1 "10k" V 7155 2000 40  0000 C CNB
+F 2 "mmM:r_0805" V 7255 2000 40  0001 C CNN
+F 3 "" H 7150 2000 40  0001 C CNN
+F 4 "RMCF0805JT10K0" H 7150 2000 40  0001 C CNN "manf#"
 	1    7150 2000
 	1    0    0    -1
@@
 U 1 1 50E2955A
 P 4175 2775
-F 0 "C23" H 4175 2875 50  0000 L CNN
-F 1 "100nF" V 4250 2450 50  0000 L CNN
-F 2 "mmM:c_0805" H 4175 2775 50  0001 C CNN
-F 3 "" H 4175 2775 60  0001 C CNN
-F 4 "CL21B104KCC5PNC" H 4175 2775 60  0001 C CNN "manf#"
+F 0 "C23" H 4200 2850 40  0000 L CNB
+F 1 "100nF" V 4225 2525 40  0000 L CNB
+F 2 "mmM:c_0805" H 4175 2775 40  0001 C CNN
+F 3 "" H 4175 2775 40  0001 C CNN
+F 4 "CL21B104KCC5PNC" H 4175 2775 40  0001 C CNN "manf#"
 	1    4175 2775
 	1    0    0    -1
@@
 U 1 1 50E29191
 P 3525 2825
-F 0 "BT2" V 3400 2600 50  0000 L CNN
-F 1 "BATT_COIN" H 3525 2635 50  0000 L CNN
-F 2 "" H 3525 2825 60  0001 C CNN
-F 3 "" H 3525 2825 60  0001 C CNN
-F 4 "CR2032" H 3525 3125 60  0001 L CNN "manf#"
+F 0 "BT2" V 3400 2600 40  0000 L CNB
+F 1 "BATT_COIN" H 3525 2625 40  0000 L CNB
+F 2 "" H 3525 2825 40  0001 C CNN
+F 3 "" H 3525 2825 40  0001 C CNN
+F 4 "CR2032" H 3525 3125 40  0001 L CNN "manf#"
 	1    3525 2825
 	0    1    1    0
@@
 U 1 1 50E29166
 P 3950 2800
-F 0 "BT1" V 3850 2625 50  0000 L CNN
-F 1 "BATT_HOLDER" H 3975 2675 50  0000 L CNN
-F 2 "mmM:CR2032" H 3950 2900 60  0001 L CNN
-F 3 "" H 3950 2800 60  0001 C CNN
-F 4 "3003" H 3950 3100 60  0001 L CNN "manf#"
+F 0 "BT1" V 3850 2675 40  0000 L CNB
+F 1 "BATT_HOLDER" H 3975 2700 40  0000 L CNB
+F 2 "mmM:CR2032" H 3950 2900 40  0001 L CNN
+F 3 "" H 3950 2800 40  0001 C CNN
+F 4 "3003" H 3950 3100 40  0001 L CNN "manf#"
 	1    3950 2800
 	0    1    1    0
@@
 Text Label 8000 4350 0    40   ~ 0
 BAT
-Text HLabel 9050 4800 2    60   Input ~ 0
+Text HLabel 9050 4800 2    40   Input ~ 0
 RST
-Text HLabel 9050 4650 2    60   Input ~ 0
+Text HLabel 9050 4650 2    40   Input ~ 0
 SQR
-Text HLabel 9050 4500 2    60   Input ~ 0
+Text HLabel 9050 4500 2    40   Input ~ 0
 32k
-Text HLabel 9050 4350 2    60   Input ~ 0
+Text HLabel 9050 4350 2    40   Input ~ 0
 BAT
 $Comp
-L +BATT #PWR16
+L +BATT #PWR019
 U 1 1 4EC101F0
 P 5300 1850
-F 0 "#PWR16" H 5300 1800 20  0001 C CNN
+F 0 "#PWR019" H 5300 1800 20  0001 C CNN
 F 1 "+BATT" H 5300 1950 30  0000 C CNN
-F 2 "" H 5300 1850 60  0001 C CNN
-F 3 "" H 5300 1850 60  0001 C CNN
+F 2 "" H 5300 1850 40  0001 C CNN
+F 3 "" H 5300 1850 40  0001 C CNN
 	1    5300 1850
 	1    0    0    -1
 $EndComp
-Text HLabel 9050 4125 2    60   Input ~ 0
+Text HLabel 9050 4125 2    40   Input ~ 0
 GND
-Text HLabel 9050 4000 2    60   Input ~ 0
+Text HLabel 9050 4000 2    40   Input ~ 0
 SDA
-Text HLabel 9050 3875 2    60   Input ~ 0
+Text HLabel 9050 3875 2    40   Input ~ 0
 SCL
-Text HLabel 9050 3750 2    60   Input ~ 0
+Text HLabel 9050 3750 2    40   Input ~ 0
 5V0
 Text Label 8050 3750 0    40   ~ 0
@@
 F 0 "B3" H 7730 2750 40  0000 L CNN
 F 1 "I_O" H 7650 2805 30  0001 C CNN
-F 2 "mmM:I_O" H 7650 2750 60  0001 C CNN
-F 3 "" H 7650 2750 60  0001 C CNN
+F 2 "mmM:I_O" H 7650 2750 40  0001 C CNN
+F 3 "" H 7650 2750 40  0001 C CNN
 	1    7650 2750
 	1    0    0    -1
@@
 F 0 "B2" H 7730 2600 40  0000 L CNN
 F 1 "I_O" H 7650 2655 30  0001 C CNN
-F 2 "mmM:I_O" H 7650 2600 60  0001 C CNN
-F 3 "" H 7650 2600 60  0001 C CNN
+F 2 "mmM:I_O" H 7650 2600 40  0001 C CNN
+F 3 "" H 7650 2600 40  0001 C CNN
 	1    7650 2600
 	1    0    0    -1
@@
 F 0 "B1" H 7730 2450 40  0000 L CNN
 F 1 "I_O" H 7650 2505 30  0001 C CNN
-F 2 "mmM:I_O" H 7650 2450 60  0001 C CNN
-F 3 "" H 7650 2450 60  0001 C CNN
+F 2 "mmM:I_O" H 7650 2450 40  0001 C CNN
+F 3 "" H 7650 2450 40  0001 C CNN
 	1    7650 2450
 	1    0    0    -1
@@
 Text Label 6500 2750 0    40   ~ 0
 32k
+Wire Bus Line
+	8000 1675 4375 1675
+Wire Bus Line
+	6575 3750 3950 3750
 $EndSCHEMATC
